File: PCB/Spikeling 3.0/Spikeling_v3.0.kicad_pcb (KiCad board)
At the start: 2 copper layers, 120 x 80 mm, 108 parts, among them J1 Connector, USB-TYPE-C-16P, J2 PJ-320B贴片, J3 PJ-320B贴片, J4 PJ-320B贴片, J5 PJ-320B贴片, J6 PJ-320B贴片, Q1 FS8205A, Q2 SI2309CDS-T1-GE3, SW1 Tactile Button, 160gf, SW2 SKHHLVA010, SW3 SKHHLVA010, SW4 SKHHLVA010, SW5 SW_Nidec_CAS-120A1, U1 ESP32-S3-WROOM-1-N4, U2 AMS1117, U3 MCP3208T-CI/SL, U4 MCP3208T-CI/SL, U5 OPA380AIDGKR, U6 MCP73812T-420I/OT, U7 BQ29700DSER, U8 TPS61200DRCR

Commit message: update PCB
Parts:
- removed .: Spikeling_neuron, Audio_Module:Spikeling_Photoreceptor
- removed .: Spikeling_neuron, Audio_Module:Spikeling_Neuron
- removed C15: 4.7uF, PCM_JLCPCB:C_0603
- removed the D2 at (159.0, 63.5)
- removed the D3 at (162.0, 63.5)
- removed the D4 at (156.2, 60.4)
- removed D9: 1SS389, PCM_JLCPCB:D_SOD-523
- removed the R14 at (133.0, 69.0)
- removed the R14 at (141.0, 69.0)
- removed REF**: Spikeling_neuron, Audio_Module:Spikeling_Electrode
- added C19: 1nF, PCM_JLCPCB:C_0603, F.Cu at (166.9, 51.4)
- added C20: 100nF, PCM_JLCPCB:C_0603, F.Cu at (133.6, 65.5)
- added C21: 10uF, PCM_JLCPCB:C_0603, F.Cu at (128.3, 67.2)
- added C22: 100nF, PCM_JLCPCB:C_0603, F.Cu at (128.3, 65.5)
- added C23: 100nF, PCM_JLCPCB:C_0603, F.Cu at (128.3, 70.5)
- added C25: 22uF, PCM_JLCPCB:C_0603, F.Cu at (128.3, 68.8)
- added R14: 1MΩ, PCM_JLCPCB:R_0603, F.Cu at (128.4, 63.8)
- added R20: 1MΩ, PCM_JLCPCB:R_0603, F.Cu at (167.0, 52.7)
- added R21: 100Ω, PCM_JLCPCB:R_0603, F.Cu at (137.7, 58.7)
- added R22: 100kΩ, PCM_JLCPCB:R_0603, F.Cu at (137.7, 60.4)
- added R23: 100Ω, PCM_JLCPCB:R_0603, F.Cu at (137.7, 63.8)
- added R24: 100kΩ, PCM_JLCPCB:R_0603, F.Cu at (137.7, 62.1)
- added R25: 100kΩ, PCM_JLCPCB:R_0603, F.Cu at (120.4, 63.8)
- added R26: 100Ω, PCM_JLCPCB:R_0603, F.Cu at (128.4, 58.7)
- added R28: 330kΩ, PCM_JLCPCB:R_0603, F.Cu at (120.4, 62.1)
- added TV1: SRV05-4-P-T7, Maxime:SOT-23-6_L2.9-W1.6-P0.95-LS2.8-BR, F.Cu at (160.5, 62.0)
- added U10: LM66100DCKR, Maxime:SC-70-6_L2.0-W1.3-P0.65-LS2.1-BL, F.Cu at (151.2, 62.0)
- added U12: LM66100DCKR, Maxime:SC-70-6_L2.0-W1.3-P0.65-LS2.1-BL, F.Cu at (124.0, 70.2)
- added U9: MF-MSMF050-2, Maxime:F1812, F.Cu at (152.0, 58.5)
- C1, C3: footprint PCM_JLCPCB:C_1206 -> PCM_JLCPCB:C_0603
- C4: footprint PCM_JLCPCB:C_0402 -> PCM_JLCPCB:C_0603
- D1: value 1N5817WS -> SMF6.0AQ; footprint Maxime:SOD-323_L1.8-W1.3-LS2.5-RD -> PCM_JLCPCB:D_SOD-123FL
- Q1: footprint Package_TO_SOT_SMD:SOT-23-6 -> Maxime:SOT-23-6_L2.9-W1.6-P0.95-LS2.8-BR
- Q2: value SI2309CDS-T1-GE3 -> P-MOSFET
- R15: value 10kΩ -> 100Ω
- R16: value 2MΩ -> 180kΩ
- R17: value 180kΩ -> 100kΩ
- R19: value 330Ω -> 1kΩ
- moved C4 32.3 mm to (120.2, 92.0)
- moved C2 29.8 mm to (133.0, 87.3)
- moved U2 28.5 mm to (126.9, 89.6)
- moved C3 28.4 mm to (120.2, 90.3)
- moved R6 26.2 mm to (120.2, 93.7), turned to 0 degrees
- moved C1 24.1 mm to (120.2, 88.6)
- moved Q2 20.3 mm to (124.4, 59.4)
- moved R15 19.5 mm to (137.7, 65.5)
- moved Q1 14.1 mm to (133.5, 61.4), turned to 180 degrees
- moved R17 13.3 mm to (128.4, 60.4), turned to 0 degrees
- moved C17 13.2 mm to (128.3, 72.2), turned to 0 degrees
- moved D1 13.0 mm to (143.0, 58.5), turned to 180 degrees
- moved C18 10.8 mm to (137.7, 70.6), turned to 0 degrees
- moved R16 10.1 mm to (128.4, 62.1)
- moved R15 9.99 mm to (133.5, 63.8), turned to 180 degrees
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- renumbered D5 to D2, D6 to D3, D7 to D4, D8 to D5, D10 to D7
Connections:
- BT1 pad 2: GNDREF -> Net-(BT1--)
- C17 pad 1: +5V -> Net-(U12-VIN)
- D1 pad 1: Net-(D1-Pad1) -> VBUS
- D1 pad 2: Net-(D1-Pad2) -> GNDREF
- J1 pad A9B4: Net-(D1-Pad2) -> Net-(J1-VBUS-PadA9B4)
- J1 pad B9A4: Net-(D1-Pad2) -> Net-(J1-VBUS-PadA9B4)
- J1 pad S1: GNDREF -> Net-(J1-SHIELD)
- L1 pad 1: Net-(D1-Pad1) -> Net-(U10-VOUT)
- L1 pad 2: VBUS -> +5V
- Q1 pad 3: GNDREF -> Net-(BT1--)
- Q2 pad 1: VBUS -> Net-(Q2-G)
- R1 pad 1: Net-(J1-CC1) -> GNDREF
- R1 pad 2: GNDREF -> Net-(J1-CC1)
- R15 pad 1: GNDREF -> Net-(U7-V-)
- R15 pad 2: Net-(SW5-A) -> Net-(Q1-D1/D2-Pad2)
- R16 pad 2: Net-(U8-FB) -> Net-(U8-UVLO)
- R17 pad 1: Net-(U8-FB) -> Net-(U8-UVLO)
- R18 pad 1: Net-(SW5-A) -> Net-(U12-ST)
- R2 pad 1: Net-(J1-CC2) -> GNDREF
- R2 pad 2: GNDREF -> Net-(J1-CC2)
- TP3 pad 1: unconnected-(TP3-Pad1) -> Pack+
- U7 pad 2: Net-(Q1-G1) -> Net-(U7-COUT)
- U7 pad 3: Net-(Q1-G2) -> Net-(U7-DOUT)
- U8 pad 2: +5V -> Net-(U12-VIN)
- U8 pad 7: Net-(SW5-A) -> Net-(U8-UVLO)
Routing:
- net +5V: track 3.00 -> 84.3 mm, vias 0 -> 2
- net Net-(J1-SHIELD): track 0.00 -> 50.9 mm
- net Net-(U12-ST): track 0.00 -> 44.5 mm
- net Net-(C1-Pad1): track 32.6 -> 74.1 mm
- net Net-(U12-VIN): track 0.00 -> 28.2 mm
- net VBUS: track 47.0 -> 25.1 mm, vias 0 -> 2
- net En: track 120.9 -> 99.5 mm
- net Net-(Q2-D): track 31.8 -> 11.8 mm
- net Net-(U7-DOUT): track 0.00 -> 19.4 mm
- net Net-(J1-VBUS-PadA9B4): track 0.00 -> 19.0 mm
- net +3.3V: track 599.6 -> 618.2 mm
- net GNDREF: track 75.3 -> 92.5 mm, vias 79 -> 129
- net Net-(U7-BAT): track 20.4 -> 4.62 mm, vias 2 -> 0
- net Net-(U7-COUT): track 0.00 -> 14.4 mm
- net Net-(U6-PROG): track 19.5 -> 5.50 mm
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Other:
- board text added: "Bat"
- board text added: "Buzzer"
- board text added: "LED"
- board text added: "Reset"
