File: PCB/Spikeling 3.0/Spikeling_v3.0.kicad_sch (KiCad schematic)
At the start: 87 parts, among them J1 Connector, USB-TYPE-C-16P, J2 PJ-320B贴片, J3 PJ-320B贴片, J4 PJ-320B贴片, J5 PJ-320B贴片, J6 PJ-320B贴片, Q1 FS8205A, Q2 SI2309CDS-T1-GE3, SW1 Tactile Button, 160gf, SW2 SKHHLVA010, SW3 SKHHLVA010, SW4 SKHHLVA010, SW5 SW_Nidec_CAS-120A1, U1 ESP32-S3-WROOM-1-N4, U2 AMS1117, U3 MCP3208T-CI/SL, U4 MCP3208T-CI/SL, U5 OPA380AIDGKR, U6 MCP73812T-420I/OT, U7 BQ29700DSER, U8 TPS61200DRCR

Commit message: update PCB
Parts:
- removed C1, C3: 22uF, PCM_JLCPCB:C_1206, symbol PCM_JLCPCB-Capacitors:1206,22uF
- removed C15: 4.7uF, PCM_JLCPCB:C_0603, symbol PCM_JLCPCB-Capacitors:0603,4.7uF
- removed C4: 100nF, PCM_JLCPCB:C_0402, symbol PCM_JLCPCB-Capacitors:0402,100nF
- removed D1: 1N5817WS, Maxime:SOD-323_L1.8-W1.3-LS2.5-RD, symbol 1N5817WS1_1N5817WS-altium-import:root_0_1N5817WS_
- removed D2, D3, D4: LESD5D5.0CT1G, Maxime:SOD-523_L1.2-W0.8-LS1.6-BI, symbol LESD5D5.0CT1G1_LESD5D5.0CT1G-altium-import:root_0_LESD5D5.0CT1G_
- removed D9: 1SS389, PCM_JLCPCB:D_SOD-523, symbol PCM_JLCPCB-Diodes:Schottky,1SS389
- removed R14: 100kΩ, PCM_JLCPCB:R_0603, symbol PCM_JLCPCB-Resistors:0603,100kΩ
- removed R15: 2.2kΩ, PCM_JLCPCB:R_0603, symbol PCM_JLCPCB-Resistors:0603,2.2kΩ
- removed R16: 2MΩ, PCM_JLCPCB:R_0603, symbol PCM_JLCPCB-Resistors:0603,2MΩ
- removed R17: 180kΩ, PCM_JLCPCB:R_0603, symbol PCM_JLCPCB-Resistors:0603,180kΩ
- removed R19: 330Ω, PCM_JLCPCB:R_0603, symbol PCM_JLCPCB-Resistors:0603,330Ω
- added C1, C25, C3: 22uF, PCM_JLCPCB:C_0603, symbol PCM_JLCPCB-Capacitors:0603,22uF
- added C19: 1nF, PCM_JLCPCB:C_0603, symbol PCM_JLCPCB-Capacitors:0603,1nF
- added C20, C22, C23, C4: 100nF, PCM_JLCPCB:C_0603, symbol PCM_JLCPCB-Capacitors:0603,100nF
- added C21: 10uF, PCM_JLCPCB:C_0603, symbol PCM_JLCPCB-Capacitors:0603,10uF
- added D1: SMF6.0AQ, PCM_JLCPCB:D_SOD-123FL, symbol PCM_JLCPCB-Diodes:TVS-Uni,SMF5.0A
- added R14, R20: 1MΩ, PCM_JLCPCB:R_0603, symbol PCM_JLCPCB-Resistors:0603,1MΩ
- added R15, R21, R23, R26: 100Ω, PCM_JLCPCB:R_0603, symbol PCM_JLCPCB-Resistors:0603,100Ω
- added R16: 180kΩ, PCM_JLCPCB:R_0603, symbol PCM_JLCPCB-Resistors:0603,180kΩ
- added R17, R22, R24, R25: 100kΩ, PCM_JLCPCB:R_0603, symbol PCM_JLCPCB-Resistors:0603,100kΩ
- added R19: 1kΩ, PCM_JLCPCB:R_0603, symbol PCM_JLCPCB-Resistors:0603,1kΩ
- added R28: 330kΩ, PCM_JLCPCB:R_0603, symbol PCM_JLCPCB-Resistors:0603,330kΩ
- added TV1: SRV05-4-P-T7, SOT-23-6_L2.9-W1.6-P0.95-LS2.8-BR, symbol SRV05-4-P-T71_SRV05-4-P-T7-altium-import:root_0_SRV05-4-P-T7_C85364_
- added U10, U12: LM66100DCKR, Maxime:SC-70-6_L2.0-W1.3-P0.65-LS2.1-BL, symbol LM66100DCKR1_LM66100DCKR-altium-import:root_0_LM66100DCKR_C2869734_
- added U9: MF-MSMF050-2, Maxime:F1812, symbol MF-MSMF050-21_MF-MSMF050-2-altium-import:root_0_MF-MSMF050-2_
- B1: ADD INTO BOM yes -> (none); ALTIUM_VALUE 4kHz -> (none); CONVERT TO PCB yes -> (none); CURRENT CONSUMPTION 5mA -> (none); DATASHEET https://atta.szlcsc.com/upload/public/pdf/source/20230614/2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 -> (none); DEVICE KMTG1203 -> (none); DRIVER CIRCUITRY Passive (Externally Driven) -> (none); HEIGHT 3mm -> (none); JLCPCB PART CLASS Extended Part -> (none); LCSC PART NAME KMTG1203 工业级-压电式无源贴片蜂鸣器 -> (none); LCSC Part # (none) -> C7421651; LENGTH 12mm -> (none); MANUFACTURER KINGSTATE(志丰电子) -> (none); MANUFACTURER PART KMTG1203 -> (none); OPERATING TEMPERATURE -40℃~+120℃ -> (none); SOUND PRESSURE LEVEL(SPL) 81dB -> (none); SUPPLIER LCSC -> (none); SUPPLIER FOOTPRINT SMD,12x12mm -> (none); SUPPLIER PART C7421651 -> (none); SYMBOL KMTG1203 -> (none); TECHNOLOGY Piezoelectric -> (none); VOLTAGE - SUPPLY - -> (none); VOLTAGE RATING 5V -> (none); WIDTH 12mm -> (none)
- BT1: LCSC Part # (none) -> C265283
- D2: renamed from D5; LCSC C2286 -> (none); LCSC Part # (none) -> C2286
- D3: renamed from D6; LCSC Part # (none) -> C67891; SUPPLIER PART C67891 -> (none)
- D4: renamed from D7; LCSC Part # (none) -> C2962096; SUPPLIER PART C2962096 -> (none)
- D7: renamed from D10; LCSC C2286 -> (none); LCSC Part # (none) -> C2286
- J1: LCSC C2927039 -> (none); LCSC Part # (none) -> C2927039
- J2, J3, J4, J5, J6: LCSC Part # (none) -> C18594; SUPPLIER PART C18594 -> (none)
- L1: LCSC Part # (none) -> C85840; SUPPLIER PART C85840 -> (none)
- Q1: footprint Package_TO_SOT_SMD:SOT-23-6 -> Maxime:SOT-23-6_L2.9-W1.6-P0.95-LS2.8-BR; LCSC Part # (none) -> C908265; SUPPLIER PART C908265 -> (none)
- Q2: value SI2309CDS-T1-GE3 -> P-MOSFET; LCSC Part # (none) -> C10493; SUPPLIER PART C10493 -> (none)
- SW1: LCSC C720477 -> (none); LCSC Part # (none) -> C720477
- SW2, SW3, SW4: LCSC Part # (none) -> C110289; SUPPLIER PART C110289 -> (none)
- SW5: LCSC Part # (none) -> C92657
- U1: LCSC Part # (none) -> C2913197; SUPPLIER PART C2913197 -> (none)
- U2: LCSC C6186 -> (none); LCSC Part # (none) -> C6186
- U3, U4: LCSC Part # (none) -> C626764; SUPPLIER PART C626764 -> (none)
- U5: LCSC Part # (none) -> C2057355; SUPPLIER PART C2057355 -> (none)
- U6: LCSC Part # (none) -> C144308; SUPPLIER PART C144308 -> (none)
- U7: LCSC Part # (none) -> C183096; SUPPLIER PART C183096 -> (none)
- U8: LCSC Part # (none) -> C140320; SUPPLIER PART C140320 -> (none)
- VR1, VR2, VR4, VR5, VR6, VR7: LCSC Part # (none) -> C470316; SUPPLIER PART C470316 -> (none)
- VR3: LCSC Part # (none) -> C361173; SUPPLIER PART C361173 -> (none)
- renumbered D8 to D5
Connections:
- net +5V: now also L1.2, U12.6 (VOUT); no longer C17.1, U8.2 (VOUT)
- net GNDREF: now also R1.1, R2.1, C1.2, C19.2, C20.2, C21.2, C22.2, C23.2, C25.2, C3.2, C4.2, D1.2, R14.2, R17.2, R20.2, R25.2, TV1.2, U10.2 (GND), U10.3 (CE#), U12.2 (GND), U12.3 (CE#); no longer BT1.2 (-), J1.S1 (SHIELD), Q1.3 (S2), R1.2, R2.2
- net Pack+: now also TP3.1, R19.1
- net USB_D+: now also TV1.1
- net USB_D-: now also TV1.3
- net VBUS: now also D1.1, R26.1, U10.1 (VIN), U9.2; no longer L1.2, Q2.1 (G)
- net at L2.1, SW5.3 (A), U8.5 (VIN)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: now also C21.1, C22.1, R14.1, R16.1; no longer R18.1, U8.7 (UVLO)
- net at L1.1: now also U10.6 (VOUT)
- net at J1.A5 (CC1): now also R1.2, TV1.4; no longer R1.1
- net at R3.1, R6.2, U2.2 (VOUT)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: now also C1.1, C3.1, C4.1
- net at U8.10 (FB): now also R25.1, R28.2
- net at J1.A9B4 (VBUS), J1.B9A4 (VBUS): now also U9.1
- net at J1.B5 (CC2): now also R2.2, TV1.6; no longer R2.1
- net at Q1.6 (G1): now also R21.2, R22.2; no longer U7.2 (COUT)
- net at Q1.4 (G2): now also R23.2, R24.2; no longer U7.3 (DOUT)
- net at C18.1, U7.5 (BAT): now also R19.2
- net at U7.6 (V-): now also C20.1, R15.1
- net at Q1.2 (D1/D2), Q1.5 (D1/D2): now also R15.2, R22.1, R24.1
- new net: R18.1, U12.5 (ST)
- new net: C17.1, C23.1, C25.1, R28.1, U12.1 (VIN), U8.2 (VOUT)
- new net: R16.2, R17.1, U8.7 (UVLO)
- new net: C19.1, J1.S1 (SHIELD), R20.1
- new net: BT1.2 (-), Q1.3 (S2)
- new net: R23.1, U7.2 (COUT)
- new net: R21.1, U7.3 (DOUT)
- new net: Q2.1 (G), R26.2
- no-connect marks 23 -> 27
Other:
- moved on the sheet: BT1, C16, C17, C18, C2, C5, C6, D2, D7, J1, L1, L2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

Commit message: PCB
Parts:
- removed C11: 1nF, PCM_JLCPCB:C_0603, symbol PCM_JLCPCB-Capacitors:0603,1nF
- removed R9: 10Ω, PCM_JLCPCB:R_0603, symbol PCM_JLCPCB-Resistors:0603,10Ω
- added C15: 100nF, PCM_JLCPCB:C_0402, symbol PCM_JLCPCB-Capacitors:0402,100nF
- added R27, R29, R30, R31, R32: 100kΩ, PCM_JLCPCB:R_0603, symbol PCM_JLCPCB-Resistors:0603,100kΩ
- added U5: MCP4922-E/SL, SOIC-14_L8.7-W3.9-P1.27-LS6.0-BL, symbol MCP4922-E_SL1_MCP4922-E_SL-altium-import:root_0_MCP4922-E/SL_
- renumbered U9 to U10, U10 to U11, U5 to U6, U6 to U7, U7 to U8, U8 to U9
Connections:
- net +3.3V: now also C15.2, U5.1 (VDD), U5.11 (VREFB), U5.13 (VREFA), U5.9 (SHDN#)
- net CurrentInput: now also R32.2
- net CurrentStimulus: now also U5.10 (VOUTB); no longer U4.4 (CH3)
- net GNDREF: now also C15.1, R27.1, R29.1, R30.1, R31.1, R32.1, U5.12 (VSS), U5.8 (LDAC#)
- net MOSI: now also U5.5 (SDI)
- net Noise: now also U4.3 (CH2); no longer U4.5 (CH4)
- net PhotoDiode: now also U4.1 (CH0); no longer U3.7 (CH6)
- net PhotoGain: now also U4.2 (CH1); no longer U3.8 (CH7)
- net SCK: now also U5.4 (SCK)
- net StimulusFrequency: now also U4.5 (CH4); no longer U4.3 (CH2)
- net StimulusStrength: now also U4.4 (CH3); no longer U4.2 (CH1)
- net Synapse1_Spike: now also R27.2
- net Synapse2_Spike: now also R30.2
- net SynapseIn1: now also R29.2
- net SynapseIn2: now also R31.2
- net SynapseOut: now also U5.14 (VOUTA); no longer U4.1 (CH0)
- net SynapseOut_Spike: now also J6.2
- net CS3: now reaches U1.15 (IO3)
- net CS3: now also U5.3 (CS#)
- no-connect marks 27 -> 34
Other:
- note added: "Analog to Digital Converter"
- note added: "ESP32S3 WROOM1 N4"
- moved on the sheet: C5, C6, H1, H2, H3, H4, R4, R5, SW1, SW2, TP1, TP2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
