File: PCB/Spikeling 2.5/Spikeling_V2.5.kicad_sch (KiCad schematic)
At the start: 47 parts, among them J1 Synapse Out, J2 Synapse in 1, J3 Synapse in 2, J4 Current in, J5 Stimulus Out, SW1 Mode Button, SW2 Buzzer Button, SW3 Reset Button, U1 ESP32-DEVKITC-32D, U2 MCP3208, U3 MCP3208

Commit message: update pcb 2.5
Parts:
- removed R?: 10kΩ, RES-TH_RK09D1130C2P, symbol Spikeling_v3.0-altium-import:root_0_RK09D1130C2P_
- D1: footprint LED_THT:LED_D5.0mm-4_RGB -> LED_THT:LED_D5.0mm-4_RGB_Wide_Pins
Connections:
- net +3V3: now also C1.2, C2.2, R10.2, RV1.3, RV2.3, RV3.3, RV4.3, RV5.3, RV6.3, RV7.3, SW1.2, SW2.2, U2.15 (Vref), U2.16 (Vdd), U3.15 (Vref), U3.16 (Vdd)
- net GNDREF: now also C3.1, R4.2; no longer C3.2, R4.1
- net VCC: no longer C1.2, C2.2, R10.2, RV1.3, RV2.3, RV3.3, RV4.3, RV5.3, RV6.3, RV7.3, SW1.2, SW2.2, U2.15 (Vref), U2.16 (Vdd), U3.15 (Vref), U3.16 (Vdd)
- net at D1.2 (K): now also R4.1; no longer R4.2
- net at J1.R, R1.2: now also C3.2; no longer C3.1
- net 00 renamed CS1
- net 02 renamed CharliePlex1
- net 04 renamed CS2
- net 05 renamed CharliePlex2
- net 100 renamed VoltageMembrane
- net 101 renamed SynapseGain1
- net 102 renamed SynapseGain2
- net 103 renamed PhotoGain
- net 104 renamed StimulusStrength
- net 105 renamed StimulusFrequency
- net 106 renamed Noise
- net 107: no longer names the net of U2.8 (CH7)
- net 12 renamed Spike_BLED
- net 13 renamed Spike_Buzzer
- net 14 renamed Spike_GLED
- net 15 renamed SynapseOut_Spike
- net 16 renamed BuzzerButton
- net BuzzerButton: now also R11.1, SW2.1
- net 17: no longer names the net of U1.30 (IO17)
- net 18 renamed SCK
- net 19 renamed CharliePlex3
- net 200 renamed SynapseIn1
- net 201 renamed SynapseIn2
- net 202 renamed PhotoDiode
- net 203 renamed CurrentInput
- net 204: no longer names the net of U3.5 (CH4)
- net 205: no longer names the net of U3.6 (CH5)
- net 206: no longer names the net of U3.7 (CH6)
- net 207: no longer names the net of U3.8 (CH7)
- net 21 renamed CharliePlex4
- net 22 renamed LightStimulus
- net 23: no longer names the net of U1.21 (IO23)
- net 25 renamed SynapseOut
- net 26 renamed CurrentStimulus
- net 27 renamed Spike_RLED
- net 32 renamed MOSI
- net 33 renamed MISO
- net 34 renamed Synapse2_Spike
- net 35 renamed Synapse1_Spike
- removed net 36: R11.1, SW2.1, U1.3 (SENSOR_VP)
- net 39 renamed ModeButton
- no-connect marks 9 -> 17
Other:
- note added: "Digital to Analog Converters"
- note added: "ESP32 WROOM 32 DevKit module"
- note added: "Neuron Modes"
- note added: "Noise"
- note added: "Photo-Receptor"
- note added: "Spike Display"
- note added: "Stimulus"
- note added: "Synapse 1"
- note added: "Synapse 2"
- note added: "Synaptic output"
- note added: "Voltage Membrane"
- company: (none) -> OpenSourceNeuro
- title: (none) -> Spikeling v2.5
- moved on the sheet: BZ1, C1, C2, C3, D1, D10, D11, D12, D13, D2, D3, D4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
