File: Hardware/PCB/Spikeling 3.1/Spikeling_v3.1.kicad_pcb (KiCad board)
At the start: 2 copper layers, 120 x 80 mm, 122 parts, among them J1 Connector, USB-TYPE-C-16P, J2 PJ-320B贴片, J3 PJ-320B贴片, J4 PJ-320B贴片, J5 PJ-320B贴片, J6 PJ-320B贴片, Q1 FS8205A, Q2 P-MOSFET, SW1 Tactile Button, 160gf, SW2 SKHHLVA010, SW3 SKHHLVA010, SW4 SKHHLVA010, SW5 SW_Nidec_CAS-120A1, U1 ESP32-S3-WROOM-1-N4, U10 MF-MSMF050-2, U11 LM66100DCKR, U12 LM66100DCKR, U2 AMS1117, U3 MCP3208T-CI/SL, U4 MCP3208T-CI/SL, U5 MCP4922-E/SL, U6 OPA380AIDGKR, U7 MCP73812T-420I/OT, U8 BQ29700DSER, U9 TPS61200DRCR

Commit message: update pcb
Changed lines of the file:
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@@
 		(property "Reference" "U5"
 			(at -0.112 -4.613 90)
-			(layer "F.SilkS")
+			(layer "F.Fab")
 			(effects
 				(font
