File: Hardware/PCB/Spikeling 3.1/Spikeling_v3.1.kicad_sch (KiCad schematic)
At the start: 105 parts, among them J1 Connector, USB-TYPE-C-16P, J2 PJ-320B贴片, J3 PJ-320B贴片, J4 PJ-320B贴片, J5 PJ-320B贴片, J6 PJ-320B贴片, Q1 FS8205A, Q2 P-MOSFET, SW1 Tactile Button, 160gf, SW2 SKHHLVA010, SW3 SKHHLVA010, SW4 SKHHLVA010, SW5 SW_Nidec_CAS-120A1, U1 ESP32-S3-WROOM-1-N4, U10 MF-MSMF050-2, U11 LM66100DCKR, U12 LM66100DCKR, U2 AMS1117, U3 MCP3208T-CI/SL, U4 MCP3208T-CI/SL, U5 MCP4922-E/SL, U6 OPA380AIDGKR, U7 MCP73812T-420I/OT, U8 BQ29700DSER, U9 TPS61200DRCR

Commit message: update pcb
Connections:
- net GNDREF: no longer U8.4 (VSS)
- net at BT1.2 (-), Q1.3 (S2): now also U8.4 (VSS)
Other:
- note added: "Analog to Digital Converters"
- note added: "Digital to Analog Converter"
- note removed: "Analog to Digital Converter"
- note removed: "Digital to Analog Converters"
Changed lines of the file:
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@@
 		)
 	)
-	(text "Digital to Analog Converters"
+	(text "Analog to Digital Converters"
 		(exclude_from_sim no)
 		(at 308.61 18.415 0)
@@
 		)
 	)
-	(text "Analog to Digital Converter"
+	(text "Digital to Analog Converter"
 		(exclude_from_sim no)
 		(at 219.075 19.05 0)
@@
 	)
 	(junction
-		(at 148.844 122.936)
-		(diameter 0)
-		(color 0 0 0 0)
-	)
-	(junction
 		(at 150.495 88.646)
 		(diameter 0)
@@
 	)
 	(junction
+		(at 96.52 109.728)
+		(diameter 0)
+		(color 0 0 0 0)
+	)
+	(junction
 		(at 149.86 41.91)
 		(diameter 0)
@@
 	(wire
 		(pts
-			(xy 148.844 99.06) (xy 148.844 122.936)
-		)
-		(stroke
-			(width 0)
-			(type default)
-		)
-	)
-	(wire
-		(pts
 			(xy 233.68 153.67) (xy 237.49 153.67)
 		)
@@
 	(wire
 		(pts
+			(xy 128.27 99.06) (xy 129.54 99.06)
+		)
+		(stroke
+			(width 0)
+			(type default)
+		)
+	)
+	(wire
+		(pts
 			(xy 284.48 127) (xy 292.1 127)
 		)
@@
 	(wire
 		(pts
+			(xy 96.52 109.728) (xy 96.52 117.856)
+		)
+		(stroke
+			(width 0)
+			(type default)
+		)
+	)
+	(wire
+		(pts
 			(xy 355.6 172.72) (xy 364.49 172.72)
 		)
@@
 	(wire
 		(pts
-			(xy 148.844 122.936) (xy 150.495 122.936)
+			(xy 147.32 122.936) (xy 150.495 122.936)
 		)
 		(stroke
@@
 	(wire
 		(pts
+			(xy 129.54 99.06) (xy 129.54 109.728)
+		)
+		(stroke
+			(width 0)
+			(type default)
+		)
+	)
+	(wire
+		(pts
 			(xy 52.324 29.972) (xy 54.61 29.972)
 		)
@@
 	(wire
 		(pts
-			(xy 128.27 99.06) (xy 148.844 99.06)
-		)
-		(stroke
-			(width 0)
-			(type default)
-		)
-	)
-	(wire
-		(pts
 			(xy 57.15 68.58) (xy 62.23 68.58)
 		)
@@
 	(wire
 		(pts
-			(xy 147.32 122.936) (xy 148.844 122.936)
-		)
-		(stroke
-			(width 0)
-			(type default)
-		)
-	)
-	(wire
-		(pts
 			(xy 160.02 33.02) (xy 160.02 31.75)
 		)
@@
 	(wire
 		(pts
+			(xy 129.54 109.728) (xy 96.52 109.728)
+		)
+		(stroke
+			(width 0)
+			(type default)
+		)
+	)
+	(wire
+		(pts
 			(xy 259.08 127) (xy 269.24 127)
 		)
@@
 	(wire
 		(pts
-			(xy 96.52 108.204) (xy 96.52 117.856)
+			(xy 96.52 108.204) (xy 96.52 109.728)
 		)
 		(stroke
