File: Hardware/PCB/Spikeling 3.2/Spikeling_v3.2.kicad_pcb (KiCad board)
At the start: 2 copper layers, 120 x 80 mm, 209 parts, among them J1 PJ-320B, J2 Connector, USB-TYPE-C-16P, J3 PJ-320B, J4 PJ-320B, J5 PJ-320B, J6 PJ-320B, Q1 FS8205A, Q2 2N7002, Q3 2N7002, Q4 2N7002, SW1 SKHHLVA010, SW2 Tactile Button, 160gf, SW3 SW_Nidec_CAS-120A1, SW4 SKHHLVA010, SW5 SKHHLVA010, U1 MCP73812T-420I/OT, U10 ESP32-S3-WROOM-1-N4, U11 LM66100DCKR, U12 MCP3208T-CI/SL, U13 TLV9001IDBVR, U14 MCP3208T-CI/SL, U2 MF-MSMF050-2, U3 LM66100DCKR, U4 OPA380AIDGKR, U5 BQ29700DSER, U6 TPS7A2033PDBVR, U7 TPS62162DSGR, U8 TPS61200DRCR, U9 MCP4922-E/SL

Commit message: update hardware
Parts:
- BT1: footprint Connector_JST:JST_XH_B2B-XH-A_1x02_P2.50mm_Vertical -> Connector_JST:JST_XH_S2B-XH-A-1_1x02_P2.50mm_Horizontal
- D9: footprint LED_THT:LED_D5.0mm-4_RGB_Wide_Pins -> LED_SMD:LED_Kingbright_APFA3010_3x1.5mm_Horizontal
- J1, J3, J4, J5, J6: footprint Maxime:AUDIO-SMD_PJ-320B -> Maxime:AUDIO-SMD_HX-PJ-320A-3P-DIP
- moved BT1 28.4 mm to (118.7, 54.7)
- moved kibuzzard-699ADA5F 11.0 mm to (188.3, 124.0), turned to -90 degrees
- moved kibuzzard-699ADB2E 10.9 mm to (166.6, 124.0), turned to -90 degrees
- moved kibuzzard-699ADBE4 9.54 mm to (106.2, 88.1)
- moved kibuzzard-699ADC07 9.47 mm to (106.2, 60.2)
- moved kibuzzard-699AE09E 9.29 mm to (110.1, 124.8)
- moved kibuzzard-699ADB4A 8.50 mm to (125.3, 123.7), turned to -90 degrees
- moved D9 7.23 mm to (214.0, 124.3), turned to 0 degrees
- moved D10 3.29 mm to (207.2, 123.7)
- moved kibuzzard-699ADACE 2.20 mm to (214.0, 68.2)
- moved kibuzzard-699ADAEF 2.19 mm to (209.8, 124.1)
- moved R65 1.37 mm to (171.7, 85.4)
- moved R64 1.35 mm to (171.7, 86.8)
- moved R3 0.78 mm to (103.6, 116.8)
- moved G*** 0.70 mm to (160.0, 89.3)
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Connections:
- D9 pad 1: Net-(D9-BA) -> Net-(D9-RA)
- D9 pad 2: Net-(D9-GA) -> GNDD
- D9 pad 3: GNDD -> Net-(D9-GA)
- D9 pad 4: Net-(D9-RA) -> Net-(D9-BA)
- U10 pad 6: Stim_GLED -> Stim_BLED
- U10 pad 7: Stim_BLED -> Stim_GLED
Routing:
- net GNDD: track 189.4 -> 221.7 mm, vias 38 -> 34
- net Cell-: track 18.3 -> 48.1 mm
- net Net-(Q4-G): track 73.5 -> 51.4 mm
- net GNDA: track 129.2 -> 145.7 mm, vias 56 -> 42
- net CurrentStimulus: track 30.2 -> 42.8 mm
- net Net-(D9-GA): track 61.3 -> 70.3 mm, vias 2 -> 3
- net Net-(D9-RA): track 58.5 -> 67.1 mm, vias 2 -> 3
- net CHASSIS: track 288.3 -> 296.5 mm
- net Cell+: track 45.6 -> 53.4 mm
- net SynapseOut: track 66.0 -> 73.7 mm
- net Boost_In: track 41.0 -> 35.8 mm
- net Net-(D11-IO1): track 7.90 -> 12.1 mm
- net Net-(D9-BA): track 64.4 -> 68.6 mm, vias 2 -> 3
- net MISO: track 87.7 -> 84.1 mm
- net Net-(D3-IO1): track 53.6 -> 56.8 mm
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Other:
- board text added: "March 2026"
- board text removed: "February 2026"

Commit message: update PCB
Parts:
- removed the D5 at (153.0, 52.3)
- removed the J1 at (106.0, 124.5)
- removed JP1: Jumper, Jumper:SolderJumper-2_P1.3mm_Open_Pad1.0x1.5mm
- removed NT1: NetTie_2, NetTie:NetTie-2_SMD_Pad0.5mm
- removed the SW3 at (126.0, 52.9)
- removed the U2 at (169.9, 55.3)
- added C59: 4.7uF, JLCPCB:C_0805, F.Cu at (199.4, 106.4)
- added C60: 100nF, JLCPCB:C_0603, F.Cu at (204.4, 103.6)
- added C61: 1uF, JLCPCB:C_0805, F.Cu at (206.0, 103.7)
- added C62: 100nF, JLCPCB:C_0603, F.Cu at (174.3, 73.9)
- added C63: 10nF, JLCPCB:C_0603, F.Cu at (181.9, 88.2)
- added C64: 100nF, JLCPCB:C_0603, F.Cu at (137.8, 74.3)
- added D10: BAT54S, JLCPCB:SOT-23-3_L2.9-W1.3-P1.90-LS2.4-BR, F.Cu at (116.7, 80.8)
- added D11: TPD2E2U06DCKR, Maxime:SC-70-3_L2.0-W1.3-P0.65-LS2.1-BL, F.Cu at (106.0, 116.4)
- added D12: BAT54S, JLCPCB:SOT-23-3_L2.9-W1.3-P1.90-LS2.4-BR, F.Cu at (106.2, 112.9)
- added D18: TPD2E2U06DCKR, Maxime:SC-70-3_L2.0-W1.3-P0.65-LS2.1-BL, F.Cu at (170.8, 66.7)
- added D19: BAT54S, JLCPCB:SOT-23-3_L2.9-W1.3-P1.90-LS2.4-BR, F.Cu at (174.2, 66.7)
- added D3: Red, JLCPCB:D_0603, F.Cu at (153.0, 52.3)
- added D4: Yellow, JLCPCB:D_0603, F.Cu at (145.0, 52.3)
- added D6: BAT54S, JLCPCB:SOT-23-3_L2.9-W1.3-P1.90-LS2.4-BR, F.Cu at (116.7, 59.3)
- added D9: BAT54S, JLCPCB:SOT-23-3_L2.9-W1.3-P1.90-LS2.4-BR, F.Cu at (116.7, 87.1)
- added J2: Synapse1 In, Maxime:AUDIO-SMD_HX-PJ-320A-3P-DIP, F.Cu at (105.8, 56.0)
- added J7: Oscilloscope Output, Maxime:AUDIO-SMD_PJ-320B, B.Cu at (170.9, 56.6)
- added R73: 100Ω, JLCPCB:R_0603, F.Cu at (158.1, 72.5)
- added R74: 100Ω, JLCPCB:R_0603, F.Cu at (156.9, 72.6)
- added R75: 10kΩ, JLCPCB:R_0603, F.Cu at (217.3, 58.4)
- added R76: 1kΩ, JLCPCB:R_0603, F.Cu at (171.7, 83.0)
- added R77: 100kΩ, JLCPCB:R_0603, F.Cu at (204.4, 57.3)
- added R78: 10kΩ, JLCPCB:R_0603, F.Cu at (185.2, 52.8)
- added R79: 10kΩ, JLCPCB:R_0603, F.Cu at (197.8, 57.6)
- added R80: 100kΩ, JLCPCB:R_0603, F.Cu at (167.8, 66.1)
- added R81: 100kΩ, JLCPCB:R_0603, F.Cu at (167.8, 67.4)
- added R82: 1kΩ, JLCPCB:R_0603, F.Cu at (169.9, 69.4)
- added SW1: K3-1260D-L1, Maxime:SW-TH_K3-1260D-L1, F.Cu at (126.0, 52.9)
- added U1: MF-MSMF050-2, Maxime:F1812, F.Cu at (169.9, 55.2)
- added U15: MCP6002T-I/SN, JLCPCB:SOIC-8_L4.9-W3.9-P1.27-LS6.0-BL, F.Cu at (208.1, 97.1)
- BT1: footprint Connector_JST:JST_XH_S2B-XH-A-1_1x02_P2.50mm_Horizontal -> Connector_JST:JST_XH_B2B-XH-A_1x02_P2.50mm_Vertical
- C1, C10, C23, C27, C33, C35, C37, C44, C45, C57, C8: footprint PCM_JLCPCB:C_0603 -> JLCPCB:C_0603
- C11, C14, C2: value 4.7uF -> 1uF; footprint PCM_JLCPCB:C_0603 -> JLCPCB:C_0805
- C12, C28, C32, C51, C53, C58: value 1uF -> 100nF; footprint PCM_JLCPCB:C_0603 -> JLCPCB:C_0603
- C13: value 4.7nF -> 100nF; footprint PCM_JLCPCB:C_0603 -> JLCPCB:C_0603
- C15: value 10pF -> 4.7uF; footprint PCM_JLCPCB:C_0603 -> JLCPCB:C_0805
- C16, C17, C31, C34, C52: value 100nF -> 4.7uF; footprint PCM_JLCPCB:C_0603 -> JLCPCB:C_0805
- C18, C30, C42, C47, C49, C56: value 4.7uF -> 100nF; footprint PCM_JLCPCB:C_0603 -> JLCPCB:C_0603
- C19, C20: value 100nF -> 22uF; footprint PCM_JLCPCB:C_0603 -> JLCPCB:C_1206
- C21, C39: value 10uF -> 100nF; footprint PCM_JLCPCB:C_0603 -> JLCPCB:C_0603
- C22, C7: value 100nF -> 10uF; footprint PCM_JLCPCB:C_0603 -> JLCPCB:C_1206
- C24: footprint PCM_JLCPCB:C_0603 -> JLCPCB:C_0805
- C25, C36, C4: value 100nF -> 1uF; footprint PCM_JLCPCB:C_0603 -> JLCPCB:C_0805
- C26: value 1nF -> 1uF; footprint PCM_JLCPCB:C_0603 -> JLCPCB:C_0805
- C29, C38: value 22uF -> 4.7uF; footprint PCM_JLCPCB:C_0603 -> JLCPCB:C_0805
- C3, C6: value 10nF -> 100nF; footprint PCM_JLCPCB:C_0603 -> JLCPCB:C_0603
- C40: value 22uF -> 1uF; footprint PCM_JLCPCB:C_0603 -> JLCPCB:C_0805
- C41: value 100nF -> 10uF; footprint PCM_JLCPCB:C_0603 -> JLCPCB:C_0805
- C43: value 1uF -> 4.7nF; footprint PCM_JLCPCB:C_0603 -> JLCPCB:C_0603
- C46: value 1uF -> 10nF; footprint PCM_JLCPCB:C_0603 -> JLCPCB:C_0603
- C48, C50: value 100nF -> 10nF; footprint PCM_JLCPCB:C_0603 -> JLCPCB:C_0603
- C5: value 10nF -> 4.7uF; footprint PCM_JLCPCB:C_0603 -> JLCPCB:C_0805
- C54: value 100nF -> 10pF; footprint PCM_JLCPCB:C_0603 -> JLCPCB:C_0603
- C55: value 100nF -> 1nF; footprint PCM_JLCPCB:C_0603 -> JLCPCB:C_0603
- C9: value 1uF -> 22uF; footprint PCM_JLCPCB:C_0603 -> JLCPCB:C_1206
- D1: value SMF6.0AQ -> SMF6.0A; footprint PCM_JLCPCB:D_SOD-123FL -> JLCPCB:D_SOD-123FL
- D2: renamed from D6; footprint PCM_JLCPCB:D_0603 -> JLCPCB:D_0603
- D7: value Yellow -> BAT54S; footprint PCM_JLCPCB:D_0603 -> JLCPCB:SOT-23-3_L2.9-W1.3-P1.90-LS2.4-BR
- J1: renamed from J2; footprint PCM_JLCPCB:TYPE-C-SMD_HX-TYPE-C-16PIN -> JLCPCB:TYPE-C-SMD_HX-TYPE-C-16PIN
- J3: value PJ-320B -> Synapse2 In
- J4: value PJ-320B -> Input Current
- J5: value PJ-320B -> Stimulus Out
- J6: value PJ-320B -> Synapse Out
- L3: renamed from L2; footprint Maxime:L0805 -> JLCPCB:L_0805
- L4: footprint PCM_JLCPCB:L_0805 -> Maxime:IND-SMD_L4.4-W4.0_PHC0420
- Q2, Q3, Q4: footprint PCM_JLCPCB:Q_SOT-23 -> JLCPCB:Q_SOT-23
- R1, R23, R24, R36, R38, R39, R40, R41, R45, R47, R49, R59, R63, R67, R68: footprint PCM_JLCPCB:R_0603 -> JLCPCB:R_0603
- R10: value 1kΩ -> 5.1MΩ; footprint PCM_JLCPCB:R_0603 -> JLCPCB:R_0603
- R11, R9: value 5.1kΩ -> 100Ω; footprint PCM_JLCPCB:R_0603 -> JLCPCB:R_0603
- R12: value 1kΩ -> 2.2kΩ; footprint PCM_JLCPCB:R_0603 -> JLCPCB:R_0603
- R13: value 1kΩ -> 330Ω; footprint PCM_JLCPCB:R_0603 -> JLCPCB:R_0603
- R14: value 1kΩ -> 910kΩ; footprint PCM_JLCPCB:R_0603 -> JLCPCB:R_0603
- R15, R17, R34: value 1kΩ -> 100kΩ; footprint PCM_JLCPCB:R_0603 -> JLCPCB:R_0603
- R16: value 1kΩ -> 1MΩ; footprint PCM_JLCPCB:R_0603 -> JLCPCB:R_0603
- R18: value 10kΩ -> 1MΩ; footprint PCM_JLCPCB:R_0603 -> JLCPCB:R_0603
- R19, R20: value 5.1MΩ -> 100kΩ; footprint PCM_JLCPCB:R_0603 -> JLCPCB:R_0603
- R2: value 4.7kΩ -> 5.1kΩ; footprint PCM_JLCPCB:R_0603 -> JLCPCB:R_0603
- R21, R33: value 10kΩ -> 100kΩ; footprint PCM_JLCPCB:R_0603 -> JLCPCB:R_0603
- R22: value 100Ω -> 5.1kΩ; footprint PCM_JLCPCB:R_0603 -> JLCPCB:R_0603
- R25, R44, R66: value 100Ω -> 10kΩ; footprint PCM_JLCPCB:R_0603 -> JLCPCB:R_0603
- R26, R27: value 1kΩ -> 100Ω; footprint PCM_JLCPCB:R_0603 -> JLCPCB:R_0603
- R28: value 2.2kΩ -> 220Ω; footprint PCM_JLCPCB:R_0603 -> JLCPCB:R_0603
- R29: value 330Ω -> 220Ω; footprint PCM_JLCPCB:R_0603 -> JLCPCB:R_0603
- R3, R4, R5: value 100kΩ -> 5.1kΩ; footprint PCM_JLCPCB:R_0603 -> JLCPCB:R_0603
- R30: value 5.1kΩ -> 10kΩ; footprint PCM_JLCPCB:R_0603 -> JLCPCB:R_0603
- R31: value 5.1kΩ -> 100kΩ; footprint PCM_JLCPCB:R_0603 -> JLCPCB:R_0603
- R32: value 0Ω -> 100kΩ; footprint PCM_JLCPCB:R_0603 -> JLCPCB:R_0603
- R35: value 22Ω -> 10kΩ; footprint PCM_JLCPCB:R_0603 -> JLCPCB:R_0603
- R37: value 47Ω -> 22Ω; footprint PCM_JLCPCB:R_0603 -> JLCPCB:R_0603
- R42: value 910kΩ -> 47Ω; footprint PCM_JLCPCB:R_0603 -> JLCPCB:R_0603
- R43: value 100kΩ -> 47Ω; footprint PCM_JLCPCB:R_0603 -> JLCPCB:R_0603
- R46: value 1kΩ -> 10kΩ; footprint PCM_JLCPCB:R_0603 -> JLCPCB:R_0603
- R48: value 47Ω -> 100kΩ; footprint PCM_JLCPCB:R_0603 -> JLCPCB:R_0603
- R50: value 1MΩ -> 1kΩ; footprint PCM_JLCPCB:R_0603 -> JLCPCB:R_0603
- R51, R55: value 100kΩ -> 1kΩ; footprint PCM_JLCPCB:R_0603 -> JLCPCB:R_0603
- R52, R60, R62, R64, R65: value 100Ω -> 1kΩ; footprint PCM_JLCPCB:R_0603 -> JLCPCB:R_0603
- R53, R54: value 1MΩ -> 100kΩ; footprint PCM_JLCPCB:R_0603 -> JLCPCB:R_0603
- R56: value 5.1kΩ -> 1kΩ; footprint PCM_JLCPCB:R_0603 -> JLCPCB:R_0603
- R57, R58: value 10kΩ -> 1kΩ; footprint PCM_JLCPCB:R_0603 -> JLCPCB:R_0603
- R6: value 1kΩ -> 0Ω; footprint PCM_JLCPCB:R_0603 -> JLCPCB:R_0603
- R61: value 100Ω -> 1MΩ; footprint PCM_JLCPCB:R_0603 -> JLCPCB:R_0603
- R69, R70, R71, R72: value 10kΩ -> 100Ω; footprint PCM_JLCPCB:R_0603 -> JLCPCB:R_0603
- R7: value 100kΩ -> 4.7kΩ; footprint PCM_JLCPCB:R_0603 -> JLCPCB:R_0603
- R8: value 100kΩ -> 5.1MΩ; footprint PCM_JLCPCB:R_0603 -> JLCPCB:R_0603
- SW2: footprint PCM_JLCPCB:SW_TS-1088-AR02016 -> JLCPCB:SW_TS-1088-AR02016
- TV1: footprint Maxime:SOT-23-6_L2.9-W1.6-P0.95-LS2.8-BR -> JLCPCB:SOT-23-6_L2.9-W1.6-P0.95-LS2.8-BR
- U14: renamed from U13; footprint Maxime:SOT-23-5_L3.0-W1.7-P0.95-LS2.8-BR -> JLCPCB:SOT-23-5_L3.0-W1.7-P0.95-LS2.8-BR
- moved R59 94.9 mm to (103.6, 116.6), turned to -90 degrees
- moved C15 86.9 mm to (200.1, 60.4)
- moved C32 84.8 mm to (212.7, 94.4)
- moved R3 83.3 mm to (163.6, 59.0), turned to 180 degrees
- moved C47 73.7 mm to (126.4, 86.9)
- moved R57 72.1 mm to (126.4, 94.9)
- moved R29 71.3 mm to (212.7, 97.2), turned to -90 degrees
- moved C40 68.3 mm to (194.2, 86.8)
- moved R27 68.1 mm to (193.6, 108.6)
- moved R26 67.4 mm to (193.6, 103.5)
- moved C55 66.8 mm to (126.4, 90.8), turned to 0 degrees
- moved C38 66.2 mm to (194.2, 83.3), turned to 90 degrees
- moved R28 64.9 mm to (203.4, 95.6), turned to -90 degrees
- moved C53 64.4 mm to (143.2, 119.1), turned to -90 degrees
- moved C39 62.9 mm to (192.5, 86.5)
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- renumbered D4 to D13, D10 to D14, D9 to D15, D8 to D16, D11 to D17, D2 to D5, D3 to D8, L3 to L2, SW1 to SW3, U12 to U10, U14 to U11, U10 to U12, U4 to U13, U3 to U2, U7 to U3, U6 to U4, U1 to U5, U5 to U6, U8 to U7, U11 to U8, VR2 to VR1, VR3 to VR2, VR1 to VR3
Connections:
- C10 pad 1: VBUS -> GNDD
- C10 pad 2: GNDD -> +3.3V
- C11 pad 1: Cell+ -> GNDA
- C11 pad 2: GNDD -> +5VA
- C12 pad 1: Net-(U3-VOUT) -> GNDA
- C12 pad 2: GNDD -> +5VA
- C13 pad 1: Boot -> GNDA
- C13 pad 2: GNDD -> +3.3VA
- C14 pad 1: GNDD -> GNDA
- C14 pad 2: +5V -> +3.3VA
- C15 pad 1: Net-(D4-C) -> GNDA
- C15 pad 2: Net-(U4-OUT) -> +3.3VA
- C16 pad 1: +5V -> GNDD
- C16 pad 2: GNDD -> VBUS
- C17 pad 1: En -> GNDD
- C17 pad 2: GNDD -> Cell+
- C18 pad 1: +3.3VA -> Cell-
- C18 pad 2: GNDA -> Net-(U6-BAT)
- C19 pad 1: +3.3VA -> Boost_5V
- C19 pad 2: GNDA -> GNDD
- C2 pad 1: Net-(JP1-A) -> GNDD
- C2 pad 2: GNDD -> VBUS
- C20 pad 1: PhotoGain -> Boost_5V
- C20 pad 2: GNDA -> GNDD
- C21 pad 1: +5V -> Boost_5V
- C22 pad 1: Net-(U5-BAT) -> GNDD
- C22 pad 2: Cell- -> Boost_In
- C23 pad 1: +5V -> GNDD
- C23 pad 2: GNDD -> Boost_In
- C24 pad 1: GNDA -> Boost_En
- C24 pad 2: Net-(U6-EN) -> GNDD
- C25 pad 1: GNDA -> GNDD
- C25 pad 2: Net-(U6-EN) -> Boost_5V
- C26 pad 1: PhotoDiode -> Net-(U8-VOUT)
- C26 pad 2: GNDA -> GNDD
- C27 pad 1: GNDA -> +3.3VA
- C27 pad 2: +3.3VA -> GNDA
- C28 pad 1: GNDA -> +3.3VA
- C28 pad 2: +3.3VA -> GNDA
- C29 pad 1: +3.3V -> GNDA
- C29 pad 2: GNDD -> +3.3VA
- C3 pad 1: CurrentInput -> GNDD
- C3 pad 2: GNDA -> VBUS
- C31 pad 1: +3.3V -> +3.3VA
- C31 pad 2: GNDD -> GNDA
- C32 pad 1: GNDD -> GNDA
- C32 pad 2: Boost_UVLO -> +3.3VA
- C33 pad 1: GNDA -> +3.3VA
- C33 pad 2: +3.3VA -> GNDA
- C34 pad 1: GNDA -> +3.3VA
- C34 pad 2: +3.3VA -> GNDA
- C35 pad 1: GNDD -> +3.3VA
- C35 pad 2: Boost_5V -> GNDA
- C36 pad 1: Noise -> +3.3VA
- C37 pad 1: Boost_In -> +3.3VA
- C37 pad 2: GNDD -> GNDA
- C38 pad 1: GNDD -> +3.3VA
- C38 pad 2: Boost_5V -> GNDA
- C39 pad 1: Boost_In -> +3.3VA
- C39 pad 2: GNDD -> GNDA
- C4 pad 1: VoltageMembrane -> GNDD
- C4 pad 2: GNDA -> Net-(U2-VOUT)
- C40 pad 1: GNDD -> +3.3VA
- C40 pad 2: Boost_5V -> GNDA
- C41 pad 1: +3.3VA -> +3.3V
- C41 pad 2: GNDA -> GNDD
- C42 pad 1: +3.3VA -> +3.3V
- C42 pad 2: GNDA -> GNDD
- C43 pad 1: Boost_5V -> Boot
- C44 pad 1: StimulusStrength -> En
- C44 pad 2: GNDA -> GNDD
- C45 pad 1: StimulusFrequency -> GNDA
- C45 pad 2: GNDA -> SynapseGain1
- C46 pad 1: Net-(U11-VOUT) -> SynapseIn1
- C46 pad 2: GNDD -> GNDA
- C47 pad 2: Net-(U13-IN+) -> SynapseGain2
- C48 pad 1: GNDA -> SynapseIn2
- C48 pad 2: +3.3VA -> GNDA
- C49 pad 1: +3.3VA -> GNDA
- C49 pad 2: GNDA -> VoltageMembrane
- C5 pad 1: SynapseIn1 -> GNDD
- C5 pad 2: GNDA -> +5V
- C50 pad 2: +3.3VA -> CurrentInput
- C51 pad 2: +3.3VA -> PhotoGain
- C52 pad 1: GNDA -> +3.3VA
- C52 pad 2: +5V -> GNDA
- C53 pad 1: GNDA -> +3.3VA
- C53 pad 2: +5V -> GNDA
- C54 pad 1: Spike_Buzzer -> Net-(D13-C)
- C54 pad 2: Net-(B1-Pad1) -> Net-(U13-OUT)
- C55 pad 2: +3.3VA -> PhotoDiode
- C56 pad 1: +3.3VA -> GNDA
- C56 pad 2: GNDA -> Noise
- C57 pad 2: +3.3VA -> StimulusStrength
- C58 pad 2: +3.3VA -> StimulusFrequency
- C6 pad 1: SynapseIn2 -> GNDD
- C6 pad 2: GNDA -> +5V
- C7 pad 1: SynapseGain2 -> GNDD
- C7 pad 2: GNDA -> +5V
- C8 pad 1: SynapseGain1 -> GNDD
- C8 pad 2: GNDA -> +5V
- C9 pad 1: VBUS -> GNDD
- C9 pad 2: GNDD -> +3.3V
- D13 pad 2: Net-(D4-C) -> Net-(D13-C)
- D14 pad 1: Net-(D10-IO1) -> Net-(D14-IO1)
- D15 pad 1: Net-(D9-RA) -> Net-(D15-RA)
- D15 pad 3: Net-(D9-GA) -> Net-(D15-GA)
- D15 pad 4: Net-(D9-BA) -> Net-(D15-BA)
- D16 pad 1: Net-(D8-RA) -> Net-(D16-RA)
- D16 pad 2: Net-(D8-BA) -> Net-(D16-BA)
- D16 pad 3: Net-(D8-GA) -> Net-(D16-GA)
- D17 pad 1: Net-(D11-IO1) -> SynapseOut
- D17 pad 2: SynapseOut -> Net-(D17-IO2)
- D2 pad 2: Net-(D6-Pad2) -> Net-(D2-Pad2)
- D5 pad 1: Net-(D2-IO1) -> Net-(D5-IO1)
- D5 pad 2: Net-(D2-IO2) -> Net-(D5-IO2)
- D7 pad 1: Net-(Q3-D) -> GNDA
- D7 pad 2: Net-(D7-Pad2) -> +3.3VA
- D8 pad 1: Net-(D3-IO1) -> Net-(D8-IO1)
- D8 pad 2: Net-(D3-IO2) -> Net-(D8-IO2)
- J3 pad 2: Net-(D2-IO2) -> Net-(D8-IO1)
- J3 pad 3: Net-(D2-IO1) -> Net-(D8-IO2)
- J4 pad 2: Net-(D3-IO2) -> unconnected-(J4-R-Pad2)
- J4 pad 3: Net-(D3-IO1) -> Net-(D11-IO1)
- J5 pad 2: CurrentStimulus -> Net-(D14-IO1)
- J5 pad 3: Net-(D10-IO1) -> CurrentStimulus
- J6 pad 2: SynapseOut -> Net-(D17-IO2)
- J6 pad 3: Net-(D11-IO1) -> SynapseOut
- L1 pad 1: Net-(U3-VOUT) -> Net-(U2-VOUT)
- L3 pad 2: Net-(U6-EN) -> +5VA
- L4 pad 1: Net-(U8-L) -> Boost_In
- L4 pad 2: Boost_In -> Net-(U7-L)
- L5 pad 1: Net-(U11-VOUT) -> Net-(U8-VOUT)
- Q4 pad 3: Net-(D11-IO1) -> Net-(D17-IO2)
- R10 pad 1: Net-(R10-Pad1) -> G_DSG
- R10 pad 2: VoltageMembrane -> Cell-
- R11 pad 1: GNDD -> G_DSG
- R11 pad 2: CC2 -> Net-(U6-DOUT)
- R12 pad 1: Net-(D2-IO1) -> Net-(U6-V-)
- R12 pad 2: Synapse1_Spike -> GNDD
- R13 pad 1: Net-(D2-IO2) -> Net-(U6-BAT)
- R13 pad 2: SynapseIn1 -> Cell+
- R14 pad 1: Net-(D3-IO1) -> Boost_FB
- R14 pad 2: Synapse2_Spike -> Boost_5V
- R15 pad 1: Net-(D3-IO2) -> Boost_FB
- R15 pad 2: SynapseIn2 -> GNDD
- R16 pad 1: Net-(R16-Pad1) -> Boost_En
- R16 pad 2: SynapseGain2 -> GNDD
- R17 pad 1: Net-(R17-Pad1) -> Net-(Q2-G)
- R17 pad 2: SynapseGain1 -> VBUS
- R18 pad 1: +3.3V -> Net-(Q2-G)
- R18 pad 2: En -> GNDD
- R19 pad 1: G_CHG -> Boost_In
- R19 pad 2: GNDD -> Boost_En
- R2 pad 2: Net-(U1-PROG) -> CC1
- R20 pad 1: G_DSG -> GNDD
- R20 pad 2: Cell- -> Net-(U7-PS)
- R21 pad 1: +3.3V -> Net-(U8-VOUT)
- R21 pad 2: Boot -> Net-(U8-ST)
- R22 pad 1: Net-(U5-COUT) -> Net-(U8-VOUT)
- R22 pad 2: G_CHG -> Net-(D4-Pad2)
- R23 pad 1: G_DSG -> Net-(U8-ST)
- R23 pad 2: Net-(U5-DOUT) -> Net-(Q3-G)
- R24 pad 1: Net-(D4-C) -> GNDD
- R24 pad 2: Net-(U4-OUT) -> Net-(Q3-G)
- R25 pad 1: Boot -> CS3
- R25 pad 2: Net-(SW2-A) -> +3.3V
- R26 pad 1: Net-(R26-Pad1) -> Net-(U9-VOUTA)
- R26 pad 2: PhotoGain -> SynapseOut_preBuff
- R27 pad 1: Net-(U4-OUT) -> Net-(U9-VOUTB)
- R27 pad 2: PhotoDiode -> CurrentStimulus_preBuff
- R28 pad 1: Net-(U5-V-) -> SynapseOut
- R28 pad 2: GNDD -> Net-(U15--INA)
- R29 pad 1: Net-(U5-BAT) -> Net-(U15--INB)
- R29 pad 2: Cell+ -> CurrentStimulus
- R3 pad 1: GNDA -> GNDD
- R3 pad 2: Net-(J1-Pad2) -> CC2
- R30 pad 1: +3.3VA -> CS1
- R30 pad 2: Net-(D5-Pad2) -> +3.3V
- R31 pad 1: Net-(D6-Pad2) -> Net-(U11-CH4)
- R31 pad 2: +3.3V -> GNDA
- R32 pad 1: GNDD -> Net-(U11-CH5)
- R33 pad 1: CS3 -> Net-(U11-CH6)
- R33 pad 2: +3.3V -> GNDA
- R34 pad 1: Net-(R34-Pad1) -> Net-(U11-CH7)
- R34 pad 2: Noise -> GNDA
- R35 pad 1: USB_D- -> +3.3V
- R35 pad 2: Net-(U10-IO19) -> CS2
- R36 pad 1: USB_D+ -> USB_D-
- R36 pad 2: Net-(U10-IO20) -> Net-(U12-IO19)
- R37 pad 1: CS3 -> USB_D+
- R37 pad 2: Net-(U10-IO3) -> Net-(U12-IO20)
- R38 pad 1: CS2 -> CS3
- R38 pad 2: Net-(U10-IO9) -> Net-(U12-IO3)
- R39 pad 1: CS1 -> CS2
- R39 pad 2: Net-(U10-IO10) -> Net-(U12-IO9)
- R4 pad 1: GNDA -> Net-(D2-Pad2)
- R4 pad 2: Net-(D2-IO1) -> +3.3V
- R40 pad 1: MOSI -> CS1
- R40 pad 2: Net-(U10-IO11) -> Net-(U12-IO10)
- R41 pad 1: SCK -> MOSI
- R41 pad 2: Net-(U10-IO12) -> Net-(U12-IO11)
- R42 pad 1: Boost_FB -> SCK
- R42 pad 2: Boost_5V -> Net-(U12-IO12)
- R43 pad 1: Boost_FB -> Net-(U12-IO13)
- R43 pad 2: GNDD -> MISO
- R44 pad 1: Net-(U9-VOUTA) -> Boot
- R44 pad 2: SynapseOut -> +3.3V
- R45 pad 1: Net-(U9-VOUTB) -> Boot
- R45 pad 2: CurrentStimulus -> Net-(SW2-A)
- R46 pad 1: Net-(R46-Pad1) -> En
- R46 pad 2: StimulusStrength -> +3.3V
- R47 pad 2: StimulusFrequency -> SynapseGain1
- R48 pad 1: Net-(U10-IO13) -> Net-(D5-IO2)
- R48 pad 2: MISO -> GNDA
- R49 pad 1: Net-(Q2-G) -> Net-(D5-IO1)
- R49 pad 2: VBUS -> GNDA
- R5 pad 1: GNDA -> Net-(D3-Pad2)
- R5 pad 2: Net-(D3-IO1) -> +3.3VA
- R50 pad 1: Net-(Q2-G) -> Net-(D5-IO2)
- R50 pad 2: GNDD -> SynapseIn1
- R51 pad 1: Net-(U11-ST) -> Net-(D5-IO1)
- R51 pad 2: Net-(U11-VOUT) -> Synapse1_Spike
- R52 pad 1: Net-(U11-ST) -> Net-(R52-Pad1)
- R52 pad 2: Net-(Q3-G) -> SynapseGain2
- R53 pad 1: Net-(Q3-G) -> Net-(D8-IO2)
- R53 pad 2: GNDD -> GNDA
- R54 pad 1: Boost_En -> Net-(D8-IO1)
- R54 pad 2: GNDD -> GNDA
- R55 pad 1: Boost_In -> Net-(D8-IO2)
- R55 pad 2: Boost_En -> SynapseIn2
- R56 pad 1: Net-(D7-Pad2) -> Net-(D8-IO1)
- R56 pad 2: Net-(U11-VOUT) -> Synapse2_Spike
- R57 pad 1: LightStimulus -> Net-(R57-Pad1)
- R57 pad 2: Net-(U13-IN+) -> VoltageMembrane
- R58 pad 1: CS1 -> Net-(D11-IO1)
- R58 pad 2: +3.3V -> CurrentInput
- R59 pad 1: GNDA -> Net-(D11-IO1)
- R59 pad 2: Net-(U13-IN+) -> GNDA
- R6 pad 1: Net-(J1-Pad2) -> GNDA
- R6 pad 2: CurrentInput -> GNDD
- R60 pad 1: Spike_BLED -> Net-(R60-Pad1)
- R60 pad 2: Net-(D8-BA) -> PhotoGain
- R61 pad 1: Spike_GLED -> Net-(D13-C)
- R61 pad 2: Net-(D8-GA) -> Net-(U13-OUT)
- R62 pad 1: Spike_RLED -> Net-(U13-OUT)
- R62 pad 2: Net-(D8-RA) -> PhotoDiode
- R63 pad 1: SynapseOut_Spike -> Net-(R63-Pad1)
- R63 pad 2: Net-(Q4-G) -> Noise
- R64 pad 1: Stim_BLED -> Net-(R64-Pad1)
- R64 pad 2: Net-(D9-BA) -> StimulusStrength
- R65 pad 1: Stim_GLED -> Net-(R65-Pad1)
- R65 pad 2: Net-(D9-GA) -> StimulusFrequency
- R66 pad 1: Stim_RLED -> Net-(U14-IN+)
- R66 pad 2: Net-(D9-RA) -> LightStimulus
- R67 pad 2: Net-(Q4-G) -> Net-(U14-IN+)
- R68 pad 1: Net-(D10-IO1) -> LightStimulus_Buff
- R68 pad 2: Net-(U13-IN-) -> Net-(D14-IO1)
- R69 pad 1: BuzzerButton -> Stim_BLED
- R69 pad 2: GNDD -> Net-(D15-BA)
- R7 pad 1: GNDA -> Net-(U5-PROG)
- R7 pad 2: Net-(D2-IO2) -> GNDD
- R70 pad 1: LEDButton -> Stim_GLED
- R70 pad 2: GNDD -> Net-(D15-GA)
- R71 pad 1: +3.3V -> Stim_RLED
- R71 pad 2: Net-(D11-IO1) -> Net-(D15-RA)
- R72 pad 1: CS2 -> Spike_BLED
- R72 pad 2: +3.3V -> Net-(D16-BA)
- R8 pad 1: GNDA -> G_CHG
- R8 pad 2: Net-(D3-IO2) -> GNDD
- R9 pad 1: GNDD -> G_CHG
- R9 pad 2: CC1 -> Net-(U6-COUT)
- U10 pad 1: SynapseGain2 -> SynapseGain1
- U10 pad 2: SynapseIn2 -> SynapseIn1
- U10 pad 3: SynapseGain1 -> SynapseGain2
- U10 pad 4: SynapseIn1 -> SynapseIn2
- U11 pad 4: unconnected-(U14-CH3-Pad4) -> OscilloscopeStimulus
- U11 pad 5: unconnected-(U14-CH4-Pad5) -> Net-(U11-CH4)
- U11 pad 6: unconnected-(U14-CH5-Pad6) -> Net-(U11-CH5)
- U11 pad 7: unconnected-(U14-CH6-Pad7) -> Net-(U11-CH6)
- U11 pad 8: unconnected-(U14-CH7-Pad8) -> Net-(U11-CH7)
- U12 pad 13: Net-(U10-IO19) -> Net-(U12-IO19)
- U12 pad 14: Net-(U10-IO20) -> Net-(U12-IO20)
- U12 pad 15: Net-(U10-IO3) -> Net-(U12-IO3)
- U12 pad 17: Net-(U10-IO9) -> Net-(U12-IO9)
- U12 pad 18: Net-(U10-IO10) -> Net-(U12-IO10)
- U12 pad 19: Net-(U10-IO11) -> Net-(U12-IO11)
- U12 pad 20: Net-(U10-IO12) -> Net-(U12-IO12)
- U12 pad 21: Net-(U10-IO13) -> Net-(U12-IO13)
- U13 pad 2: Net-(D4-C) -> Net-(D13-C)
- U13 pad 6: Net-(U4-OUT) -> Net-(U13-OUT)
- U14 pad 1: Net-(U13-IN-) -> LightStimulus_Buff
- U14 pad 3: Net-(U13-IN+) -> Net-(U14-IN+)
- U14 pad 4: Net-(U13-IN-) -> LightStimulus_Buff
- U2 pad 5: unconnected-(U3-ST-Pad5) -> GNDD
- U2 pad 6: Net-(U3-VOUT) -> Net-(U2-VOUT)
- U4 pad 1: Net-(U6-EN) -> +5VA
- U4 pad 3: Net-(U6-EN) -> +5VA
- U5 pad 1: Net-(JP1-A) -> VBUS
- U5 pad 4: Net-(JP1-A) -> VBUS
- U5 pad 5: Net-(U1-PROG) -> Net-(U5-PROG)
- U6 pad 2: Net-(U5-COUT) -> Net-(U6-COUT)
- U6 pad 3: Net-(U5-DOUT) -> Net-(U6-DOUT)
- U6 pad 5: Net-(U5-BAT) -> Net-(U6-BAT)
- U6 pad 6: Net-(U5-V-) -> Net-(U6-V-)
- U7 pad 3: Net-(U8-L) -> Net-(U7-L)
- U7 pad 8: Boost_In -> Net-(U7-PS)
- U8 pad 5: Net-(U11-ST) -> Net-(U8-ST)
- U8 pad 6: Net-(U11-VOUT) -> Net-(U8-VOUT)
- VR1 pad 2: Net-(R17-Pad1) -> Net-(R47-Pad1)
- VR2 pad 2: Net-(R16-Pad1) -> Net-(R52-Pad1)
- VR3 pad 2: Net-(R10-Pad1) -> Net-(R57-Pad1)
- VR4 pad 2: Net-(R26-Pad1) -> Net-(R60-Pad1)
- VR5 pad 2: Net-(R34-Pad1) -> Net-(R63-Pad1)
- VR6 pad 2: Net-(R46-Pad1) -> Net-(R64-Pad1)
- VR7 pad 2: Net-(R47-Pad1) -> Net-(R65-Pad1)
Routing:
- net GNDA: track 145.7 -> 274.0 mm, vias 42 -> 52
- net +3.3VA: track 647.9 -> 766.5 mm, vias 13 -> 12
- net Net-(J1-Pad2): track 73.2 -> 0.00 mm
- net Net-(D15-GA): track 0.00 -> 71.3 mm, vias 0 -> 3
- net Net-(D15-BA): track 0.00 -> 70.6 mm, vias 0 -> 3
- net Net-(D9-GA): track 70.3 -> 0.00 mm, vias 3 -> 0
- net CHASSIS: track 296.5 -> 366.6 mm
- net Net-(D2-IO1): track 70.0 -> 0.00 mm
- net Net-(D15-RA): track 0.00 -> 68.8 mm, vias 0 -> 3
- net Net-(D9-BA): track 68.6 -> 0.00 mm, vias 3 -> 0
- net Net-(D9-RA): track 67.1 -> 0.00 mm, vias 3 -> 0
- net CurrentInput: track 5.62 -> 68.0 mm
- net Synapse1_Spike: track 1.87 -> 62.5 mm
- net Net-(D3-IO1): track 56.8 -> 0.00 mm, vias 2 -> 0
- net Net-(D2-IO2): track 56.6 -> 0.00 mm, vias 2 -> 0
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Other:
- outline, holes or cut-outs redrawn
- board text added: "Buffered Analog Output"
- board text added: "USB Power"
- board text removed: "Boost Enabler"
- board text removed: "Solder here to connect LiPo battery"
- board text removed: "USB Power Entry"
- board text removed: "←"
