File: Hardware/PCB/Spikeling 3.2/Spikeling_v3.2.kicad_pcb (KiCad board)
At the start: 2 copper layers, 120 x 80 mm, 233 parts, among them J1 Connector, USB-TYPE-C-16P, J2 Synapse1 In, J3 Synapse2 In, J4 Input Current, J5 Stimulus Out, J6 Synapse Out, J7 Oscilloscope Output, Q1 FS8205A, Q2 2N7002, Q3 2N7002, Q4 2N7002, SW1 K3-1260D-L1, SW2 Tactile Button, 160gf, SW3 SKHHLVA010, SW4 SKHHLVA010, SW5 SKHHLVA010, U1 MF-MSMF050-2, U10 MCP3208T-CI/SL, U11 MCP3208T-CI/SL, U12 ESP32-S3-WROOM-1-N4, U13 OPA380AIDGKR, U14 TLV9001IDBVR, U15 MCP6002T-I/SN, U2 LM66100DCKR, U3 TPS62162DSGR, U4 TPS7A2033PDBVR, U5 MCP73812T-420I/OT, U6 BQ29700DSER, U7 TPS61200DRCR, U8 LM66100DCKR, U9 MCP4922-E/SL

Commit message: update PCB
Routing:
- net Cell-: track 46.8 -> 43.3 mm
- net +3.3V: track 607.3 -> 606.7 mm
Other:
- board text added: "+"
- board text added: "-"
