File: Hardware/PCB/Spikeling 3.2/Spikeling_v3.2.kicad_sch (KiCad schematic)
At the start: 195 parts, among them J1 PJ-320B, J2 Connector, USB-TYPE-C-16P, J3 PJ-320B, J4 PJ-320B, J5 PJ-320B, J6 PJ-320B, Q1 FS8205A, Q2 2N7002, Q3 2N7002, Q4 2N7002, SW1 SKHHLVA010, SW2 Tactile Button, 160gf, SW3 SW_Nidec_CAS-120A1, SW4 SKHHLVA010, SW5 SKHHLVA010, U1 MCP73812T-420I/OT, U10 ESP32-S3-WROOM-1-N4, U11 LM66100DCKR, U12 MCP3208T-CI/SL, U13 TLV9001IDBVR, U14 MCP3208T-CI/SL, U2 MF-MSMF050-2, U3 LM66100DCKR, U4 OPA380AIDGKR, U5 BQ29700DSER, U6 TPS7A2033PDBVR, U7 TPS62162DSGR, U8 TPS61200DRCR, U9 MCP4922-E/SL

Commit message: update hardware
Parts:
- D9: footprint LED_THT:LED_D5.0mm-4_RGB_Wide_Pins -> LED_SMD:LED_Kingbright_APFA3010_3x1.5mm_Horizontal
- J1, J3, J4, J5, J6: footprint Maxime:AUDIO-SMD_PJ-320B -> Maxime:AUDIO-SMD_HX-PJ-320A-3P-DIP
Connections:
- net GNDD: now also D9.2 (K); no longer D9.3 (K)
- net Stim_BLED: now also U10.6 (IO6); no longer U10.7 (IO7)
- net Stim_GLED: now also U10.7 (IO7); no longer U10.6 (IO6)
- net at R64.2: now also D9.4 (BA); no longer D9.1 (BA)
- net at R65.2: now also D9.3 (GA); no longer D9.2 (GA)
- net at R66.2: now also D9.1 (RA); no longer D9.4 (RA)
Other:
- moved on the sheet: D11, R71

Commit message: update PCB
Parts:
- removed C1, C26: 1nF, PCM_JLCPCB:C_0603, symbol PCM_JLCPCB-Capacitors:0603,1nF
- removed C10, C16, C17, C19, C20, C22, C23, C25, C27, C31, C33, C34, C35, C36, C37, C4, C41, C44, C45, C48, C50, C52, C54, C55, C57, C7, C8: 100nF, PCM_JLCPCB:C_0603, symbol PCM_JLCPCB-Capacitors:0603,100nF
- removed C11, C14, C18, C2, C30, C42, C47, C49, C56: 4.7uF, PCM_JLCPCB:C_0603, symbol PCM_JLCPCB-Capacitors:0603,4.7uF
- removed C12, C24, C28, C32, C43, C46, C51, C53, C58, C9: 1uF, PCM_JLCPCB:C_0603, symbol PCM_JLCPCB-Capacitors:0603,1uF
- removed C13: 4.7nF, PCM_JLCPCB:C_0603, symbol PCM_JLCPCB-Capacitors:0603,4.7nF
- removed C15: 10pF, PCM_JLCPCB:C_0603, symbol PCM_JLCPCB-Capacitors:0603,10pF
- removed C21, C39: 10uF, PCM_JLCPCB:C_0603, symbol PCM_JLCPCB-Capacitors:0603,10uF
- removed C29, C38, C40: 22uF, PCM_JLCPCB:C_0603, symbol PCM_JLCPCB-Capacitors:0603,22uF
- removed C3, C5, C6: 10nF, PCM_JLCPCB:C_0603, symbol PCM_JLCPCB-Capacitors:0603,10nF
- removed D1: SMF6.0AQ, PCM_JLCPCB:D_SOD-123FL, symbol PCM_JLCPCB-Diodes:TVS-Uni,SMF5.0A
- removed J1, J3, J4, J5, J6: PJ-320B, Maxime:AUDIO-SMD_HX-PJ-320A-3P-DIP, symbol PJ-320B1_PJ-320B-altium-import:root_0_PJ-320B贴片_
- removed JP1: Jumper, Jumper:SolderJumper-2_P1.3mm_Open_Pad1.0x1.5mm, symbol Jumper:Jumper_2_Bridged
- removed L4: 2.2uH, PCM_JLCPCB:L_0805, symbol PCM_JLCPCB-Inductors:2.2uH,50mA
- removed NT1: NetTie_2, NetTie:NetTie-2_SMD_Pad0.5mm, symbol Device:NetTie_2
- removed R1, R24, R50, R53, R54: 1MΩ, PCM_JLCPCB:R_0603, symbol PCM_JLCPCB-Resistors:0603,1MΩ
- removed R10, R12, R13, R14, R15, R16, R17, R26, R27, R34, R46, R47, R6, R63: 1kΩ, PCM_JLCPCB:R_0603, symbol PCM_JLCPCB-Resistors:0603,1kΩ
- removed R11, R30, R31, R56, R9: 5.1kΩ, PCM_JLCPCB:R_0603, symbol PCM_JLCPCB-Resistors:0603,5.1kΩ
- removed R18, R21, R33, R57, R58, R69, R70, R71, R72: 10kΩ, PCM_JLCPCB:R_0603, symbol PCM_JLCPCB-Resistors:0603,10kΩ
- removed R19, R20: 5.1MΩ, PCM_JLCPCB:R_0603, symbol PCM_JLCPCB-Resistors:0603,5.1MΩ
- removed R2: 4.7kΩ, PCM_JLCPCB:R_0603, symbol PCM_JLCPCB-Resistors:0603,4.7kΩ
- removed R22, R23, R25, R44, R45, R52, R60, R61, R62, R64, R65, R66: 100Ω, PCM_JLCPCB:R_0603, symbol PCM_JLCPCB-Resistors:0603,100Ω
- removed R28: 2.2kΩ, PCM_JLCPCB:R_0603, symbol PCM_JLCPCB-Resistors:0603,2.2kΩ
- removed R29: 330Ω, PCM_JLCPCB:R_0603, symbol PCM_JLCPCB-Resistors:0603,330Ω
- removed R3, R4, R43, R49, R5, R51, R55, R59, R67, R7, R8: 100kΩ, PCM_JLCPCB:R_0603, symbol PCM_JLCPCB-Resistors:0603,100kΩ
- removed R32: 0Ω, PCM_JLCPCB:R_0603, symbol PCM_JLCPCB-Resistors:0603,0Ω
- removed R35, R36: 22Ω, PCM_JLCPCB:R_0603, symbol PCM_JLCPCB-Resistors:0603,22Ω
- removed R37, R38, R39, R40, R41, R48: 47Ω, PCM_JLCPCB:R_0603, symbol PCM_JLCPCB-Resistors:0603,47Ω
- removed R42: 910kΩ, PCM_JLCPCB:R_0603, symbol Spikeling_V2.5-altium-import:root_0_0603WAF9103T5E_
- removed R68: 150Ω, PCM_JLCPCB:R_0603, symbol PCM_JLCPCB-Resistors:0603,150Ω
- removed SW3: SW_Nidec_CAS-120A1, Maxime:SW-TH_MMP122-R, symbol Switch:SW_Nidec_CAS-120A1
- added C1, C55: 1nF, JLCPCB:C_0603, symbol CC0603KRX7R9BB1021_CC0603KRX7R9BB102 (1)-altium-import:root_0_CC0603KRX7R9BB102_
- added C10, C12, C13, C18, C21, C23, C27, C28, C3, C30, C32, C33, C35, C37, C39, C42, C44, C45, C47, C49, C51, C53, C56, C57, C58, C6, C60, C62, C64, C8: 100nF, JLCPCB:C_0603, symbol CL10B104KB8NNNC1_CL10B104KB8NNNC (2)-altium-import:root_0_CL10B104KB8NNNC_
- added C11, C14, C2, C24, C25, C26, C36, C4, C40, C61: 1uF, JLCPCB:C_0805, symbol CL21B105KBFNNNE1_CL21B105KBFNNNE-altium-import:root_0_CL21B105KBFNNNE_
- added C15, C16, C17, C29, C31, C34, C38, C5, C52, C59: 4.7uF, JLCPCB:C_0805, symbol CS2012X7R475K350NRE1_CS2012X7R475K350NRE-altium-import:root_0_CS2012X7R475K350N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
- added C19, C20, C9: 22uF, JLCPCB:C_1206, symbol CL31A226KAHNNNE1_CL31A226KAHNNNE-altium-import:root_0_CL31A226KAHNNNE_
- added C22, C7: 10uF, JLCPCB:C_1206, symbol TCC1206X7R106K250HT1_TCC1206X7R106K250HT-altium-import:root_0_TCC1206X7R106K250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
- added C41: 10uF, JLCPCB:C_0805, symbol CL21A106KBYQNNE1_CL21A106KBYQNNE-altium-import:root_0_CL21A106KBYQNNE_
- added C43: 4.7nF, JLCPCB:C_0603, symbol 0603B472K500NT1_0603B472K500NT-altium-import:root_0_0603B472K500NT_
- added C46, C48, C50, C63: 10nF, JLCPCB:C_0603, symbol CC0603KRX7R9BB1031_CC0603KRX7R9BB103 (1)-altium-import:root_0_CC0603KRX7R9BB103_
- added C54: 10pF, JLCPCB:C_0603, symbol 0603CG100J500NT1_0603CG100J500NT-altium-import:root_0_0603CG100J500NT_
- added D1: SMF6.0A, JLCPCB:D_SOD-123FL, symbol SMF6.0A_C1782601_SMF6.0A_C178260-altium-import:root_0_SMF6.0A_C178260_
- added D10, D12, D19, D6, D7, D9: BAT54S, JLCPCB:SOT-23-3_L2.9-W1.3-P1.90-LS2.4-BR, symbol BAT54S_C9164251_BAT54S_C916425 (1)-altium-import:root_0_BAT54S_C916425_
- added D11, D18: TPD2E2U06DCKR, Maxime:SC-70-3_L2.0-W1.3-P0.65-LS2.1-BL, symbol Spikeling_V2.5-altium-import:root_0_TPD2E2U06DCKR_
- added J2: Synapse1 In, Maxime:AUDIO-SMD_HX-PJ-320A-3P-DIP, symbol HX PJ-320A-3P DIP1_HX PJ-320A-3P DIP (1)-altium-import:root_0_HX PJ-320A-3P DIP_
- added J3: Synapse2 In, Maxime:AUDIO-SMD_HX-PJ-320A-3P-DIP, symbol HX PJ-320A-3P DIP1_HX PJ-320A-3P DIP (1)-altium-import:root_0_HX PJ-320A-3P DIP_
- added J4: Input Current, Maxime:AUDIO-SMD_HX-PJ-320A-3P-DIP, symbol HX PJ-320A-3P DIP1_HX PJ-320A-3P DIP (1)-altium-import:root_0_HX PJ-320A-3P DIP_
- added J5: Stimulus Out, Maxime:AUDIO-SMD_HX-PJ-320A-3P-DIP, symbol HX PJ-320A-3P DIP1_HX PJ-320A-3P DIP (1)-altium-import:root_0_HX PJ-320A-3P DIP_
- added J6: Synapse Out, Maxime:AUDIO-SMD_HX-PJ-320A-3P-DIP, symbol HX PJ-320A-3P DIP1_HX PJ-320A-3P DIP (1)-altium-import:root_0_HX PJ-320A-3P DIP_
- added J7: Oscilloscope Output, Maxime:AUDIO-SMD_PJ-320B, symbol PJ-320B1_PJ-320B-altium-import:root_0_PJ-320B贴片_
- added L4: 2.2uH, Maxime:IND-SMD_L4.4-W4.0_PHC0420, symbol APH0420T2R2M1_APH0420T2R2M-altium-import:root_0_APH0420T2R2M_
- added R1, R16, R18, R24, R61: 1MΩ, JLCPCB:R_0603, symbol RC0603FR-071ML1_RC0603FR-071ML (1)-altium-import:root_0_RC0603FR-071ML_
- added R10, R8: 5.1MΩ, JLCPCB:R_0603, symbol AC0603FR-075M1L1_AC0603FR-075M1L-altium-import:root_0_AC0603FR-075M1L_
- added R11, R23, R26, R27, R45, R69, R70, R71, R72, R73, R74, R9: 100Ω, JLCPCB:R_0603, symbol RC0603FR-07100RL1_RC0603FR-07100RL (4)-altium-import:root_0_RC0603FR-07100RL_
- added R12: 2.2kΩ, JLCPCB:R_0603, symbol 0603WAF2201T5E1_0603WAF2201T5E-altium-import:root_0_0603WAF2201T5E_C4190_
- added R13: 330Ω, JLCPCB:R_0603, symbol 0603WAF3300T5E1_0603WAF3300T5E (1)-altium-import:root_0_0603WAF3300T5E_
- added R14: 910kΩ, JLCPCB:R_0603, symbol 0603WAF9103T5E1_0603WAF9103T5E (1)-altium-import:root_0_0603WAF9103T5E_
- added R15, R17, R19, R20, R21, R31, R32, R33, R34, R48, R49, R53, R54, R59, R67, R77, R80, R81: 100kΩ, JLCPCB:R_0603, symbol RC0603FR-07100KL1_RC0603FR-07100KL (1)-altium-import:root_0_RC0603FR-07100KL_
- added R2, R22, R3, R4, R5: 5.1kΩ, JLCPCB:R_0603, symbol 0603WAF5101T5E1_0603WAF5101T5E-altium-import:root_0_0603WAF5101T5E_
- added R25, R30, R35, R44, R46, R66, R75, R78, R79: 10kΩ, JLCPCB:R_0603, symbol FRC0603F1002TS1_FRC0603F1002TS-altium-import:root_0_FRC0603F1002TS_
- added R28, R29: 220Ω, JLCPCB:R_0603, symbol RC0603FR-07220RL1_RC0603FR-07220RL-altium-import:root_0_RC0603FR-07220RL_
- added R36, R37: 22Ω, JLCPCB:R_0603, symbol 0603WAF220JT5E1_0603WAF220JT5E-altium-import:root_0_0603WAF220JT5E_
- added R38, R39, R40, R41, R42, R43: 47Ω, JLCPCB:R_0603, symbol 0603WAF470JT5E1_0603WAF470JT5E-altium-import:root_0_0603WAF470JT5E_
- added R47, R52: 1kΩ, JLCPCB:R_0603, symbol FRC0603F1001TS1_FRC0603F1001TS (1)-altium-import:root_0_FRC0603F1001TS_
- added R50, R51, R55, R56, R57, R58, R60, R63, R64, R65, R76, R82: 1kΩ, JLCPCB:R_0603, symbol FRC0603F1001TS1_FRC0603F1001TS (2)-altium-import:root_0_FRC0603F1001TS_
- added R6: 0Ω, JLCPCB:R_0603, symbol 0603WAF0000T5E1_0603WAF0000T5E-altium-import:root_0_0603WAF0000T5E_
- added R62: 1kΩ, JLCPCB:R_0603, symbol FRC0603F1001TS1_FRC0603F1001TS-altium-import:root_0_FRC0603F1001TS_
- added R68: 150Ω, JLCPCB:R_0603, symbol 0603WAF1500T5E1_0603WAF1500T5E-altium-import:root_0_0603WAF1500T5E_
- added R7: 4.7kΩ, JLCPCB:R_0603, symbol 0603WAF4701T5E1_0603WAF4701T5E (1)-altium-import:root_0_0603WAF4701T5E_
- added SW1: K3-1260D-L1, Maxime:SW-TH_K3-1260D-L1, symbol K3-1260D-L11_K3-1260D-L1-altium-import:root_0_K3-1260D-L1_
- added U15: MCP6002T-I/SN, JLCPCB:SOIC-8_L4.9-W3.9-P1.27-LS6.0-BL, symbol MCP6002T-I_SN1_MCP6002T-I_SN-altium-import:root_0_MCP6002T-I/SN_
- D13: renamed from D4; DATASHEET https://atta.szlcsc.com/upload/public/pdf/source/20200102/C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 -> (none)
- D14: renamed from D10; DATASHEET https://www.ti.com/cn/lit/gpn/tpd2e2u06 -> (none); LCSC Part # (none) -> C1855726; SUPPLIER PART C1855726 -> (none)
- D17: renamed from D11; DATASHEET https://www.ti.com/cn/lit/gpn/tpd2e2u06 -> (none); LCSC Part # (none) -> C1855726; SUPPLIER PART C1855726 -> (none)
- D2: renamed from D6; footprint PCM_JLCPCB:D_0603 -> JLCPCB:D_0603; Manufacturer Hubei KENTO Elec -> (none)
- D3: renamed from D5; footprint PCM_JLCPCB:D_0603 -> JLCPCB:D_0603; Manufacturer Hubei KENTO Elec -> (none)
- D4: renamed from D7; footprint PCM_JLCPCB:D_0603 -> JLCPCB:D_0603; LCSC C89811 -> (none); LCSC Part # (none) -> C89811; Manufacturer Foshan NationStar Optoelectronics -> (none); Operating Temperature -30°C~+85°C -> (none)
- D5: renamed from D2; DATASHEET https://www.ti.com/cn/lit/gpn/tpd2e2u06 -> (none); LCSC Part # (none) -> C1855726; SUPPLIER PART C1855726 -> (none)
- D8: renamed from D3; DATASHEET https://www.ti.com/cn/lit/gpn/tpd2e2u06 -> (none); LCSC Part # (none) -> C1855726; SUPPLIER PART C1855726 -> (none)
- J1: renamed from J2; footprint PCM_JLCPCB:TYPE-C-SMD_HX-TYPE-C-16PIN -> JLCPCB:TYPE-C-SMD_HX-TYPE-C-16PIN
- L1, L5: DATASHEET https://atta.szlcsc.com/upload/public/pdf/source/20180326/C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 -> (none)
- L2: renamed from L3; DATASHEET https://www.coilcraft.com/getmedia/f76a3c9b-4fff-4397-8028-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 -> (none); LCSC Part # (none) -> C3911432; SUPPLIER PART C3911432 -> (none)
- L3: renamed from L2; footprint L0805 -> JLCPCB:L_0805; DATASHEET https://item.szlcsc.com/datasheet/MPZ2012S601AT000/22238.ht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 -> (none); LCSC Part # (none) -> C21519; SUPPLIER PART C21519 -> (none)
- Q1: DATASHEET https://atta.szlcsc.com/upload/public/pdf/source/20201027/C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 -> (none)
- Q2, Q3, Q4: footprint PCM_JLCPCB:Q_SOT-23 -> JLCPCB:Q_SOT-23; Gate Threshold Voltage (Vgs(th)@Id) 2.5V@250uA -> (none); LCSC C8545 -> (none); LCSC Part # (none) -> C8545; Manufacturer Changjiang Electronics Tech (CJ) -> (none); Operating Temperature -55°C~+150°C -> (none); Reverse Transfer Capacitance (Crss@Vds) 5pF -> (none); Type 1 N-channel -> (none)
- SW2: footprint PCM_JLCPCB:SW_TS-1088-AR02016 -> JLCPCB:SW_TS-1088-AR02016; Actuator Style Round Button -> (none); Circuit SPST -> (none); Contact Current 50mA -> (none); Manufacturer XUNPU -> (none); Mechanical Life 100000 Times -> (none); Mounting Style Brick nogging -> (none); Operating Temperature -30°C~+80°C -> (none); Switch Height 2mm -> (none); Switch Length 4mm -> (none); Switch Width 3mm -> (none); Voltage Rating (Dc) 12V -> (none); With Lamp No -> (none)
- SW3: renamed from SW1; DATASHEET https://atta.szlcsc.com/upload/public/pdf/source/20170428/1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 -> (none); LCSC Part # C110289 -> C2845277
- SW4, SW5: DATASHEET https://atta.szlcsc.com/upload/public/pdf/source/20170428/1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 -> (none); LCSC Part # C110289 -> C2845277
- TV1: footprint SOT-23-6_L2.9-W1.6-P0.95-LS2.8-BR -> JLCPCB:SOT-23-6_L2.9-W1.6-P0.95-LS2.8-BR; DATASHEET https://item.szlcsc.com/datasheet/SRV05-4-P-T7/86537.html -> (none)
- U1: renamed from U2; DATASHEET https://item.szlcsc.com/datasheet/MF-MSMF050-2/17998.html -> (none)
- U10: renamed from U12; DATASHEET https://atta.szlcsc.com/upload/public/pdf/source/20140724/1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 -> (none)
- U11: renamed from U14; DATASHEET https://atta.szlcsc.com/upload/public/pdf/source/20140724/1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 -> (none)
- U12: renamed from U10; DATASHEET https://atta.szlcsc.com/upload/public/pdf/source/20241030/6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 -> (none)
- U13: renamed from U4; DATASHEET https://www.ti.com/cn/lit/gpn/opa380 -> (none)
- U14: renamed from U13; footprint SOT-23-5_L3.0-W1.7-P0.95-LS2.8-BR -> JLCPCB:SOT-23-5_L3.0-W1.7-P0.95-LS2.8-BR; DATASHEET https://www.ti.com/cn/lit/gpn/tlv9001 -> (none); LCSC Part # (none) -> C398363; SUPPLIER PART C398363 -> (none)
- U2: renamed from U3; DATASHEET https://www.ti.com/cn/lit/gpn/lm66100 -> (none)
- U3: renamed from U7; DATASHEET https://www.ti.com/cn/lit/gpn/tps62162 -> (none); LCSC Part # (none) -> C40256; SUPPLIER PART C40256 -> (none)
- U4: renamed from U6; DATASHEET https://www.ti.com/cn/lit/gpn/tps7a20 -> (none); LCSC Part # (none) -> C2862740; SUPPLIER PART C2862740 -> (none)
- U5: renamed from U1; DATASHEET https://atta.szlcsc.com/upload/public/pdf/source/20171212/C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 -> (none)
- U6: renamed from U5; DATASHEET https://www.ti.com/cn/lit/gpn/bq2970 -> (none)
- U7: renamed from U8; DATASHEET https://www.ti.com/cn/lit/gpn/tps61200 -> (none)
- U8: renamed from U11; DATASHEET https://www.ti.com/cn/lit/gpn/lm66100 -> (none)
- U9: DATASHEET https://item.szlcsc.com/datasheet/MCP4922-E%252FSL/40833.ht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 -> (none); LCSC Part # (none) -> C39851; SUPPLIER PART C39851 -> (none)
- VR1: renamed from VR2; DATASHEET https://atta.szlcsc.com/upload/public/pdf/source/20191216/C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 -> (none)
- VR2: renamed from VR3; DATASHEET https://atta.szlcsc.com/upload/public/pdf/source/20191216/C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 -> (none)
- VR3: renamed from VR1; DATASHEET https://atta.szlcsc.com/upload/public/pdf/source/20191216/C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 -> (none)
- VR4, VR6, VR7: DATASHEET https://atta.szlcsc.com/upload/public/pdf/source/20191216/C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 -> (none)
- VR5: DATASHEET https://atta.szlcsc.com/upload/public/pdf/source/20190109/C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 -> (none)
- renumbered D9 to D15, D8 to D16
Connections:
- net +3.3V: now also C10.2, C41.1, C42.1, C9.2, R25.2, R30.2, R35.1, R4.2, R44.2, R46.2, R75.1
- net +3.3VA: now also C13.2, C14.2, C15.2, C27.1, C28.1, C29.2, C30.2, C31.1, C32.2, C33.1, C34.1, C35.1, C36.1, C37.1, C38.1, C39.1, C40.1, C52.1, C53.1, D10.2 (K), D12.2 (K), D19.2 (K), D6.2 (K), D7.2 (K), D9.2 (K), R5.2, U15.8 (VDD)
- net +5V: now also C5.2, C6.2, C60.2, C61.2, C7.2, C8.2
- net Boost_5V: now also C19.1, C20.1, C21.1, C25.2, R14.2
- net Boost_En: now also C24.1, R16.1, R19.2
- net Boost_FB: now also R14.1, R15.1
- net Boost_In: now also C22.2, C23.2, L4.1, R19.1, SW1.1; no longer U7.8 (PS)
- net Boost_UVLO: now also C64.1
- net Boot: now also C43.1, R44.1, R45.1
- net BuzzerButton: now also R78.1
- net CC1: now also R2.2
- net CC2: now also R3.2
- net CHASSIS: now also C1.1, R1.1
- net CS1: now also R30.1, R40.1
- net CS2: now also R35.2, R39.1
- net CS3: now also R25.1, R38.1
- net Cell+: now also C17.2, R13.2, SW1.2
- net Cell-: now also C18.1, R10.2
- net CurrentInput: now also C50.2, D12.3, R58.2
- net CurrentStimulus: now also J5.3 (T), R29.2
- net En: now also C44.1, R46.1
- net GNDA: now also C11.1, C12.1, C13.1, C14.1, C15.1, C27.2, C28.2, C29.1, C30.1, C31.2, C32.1, C33.2, C34.2, C35.2, C36.2, C37.2, C38.2, C39.2, C40.2, C45.1, C46.2, C47.1, C48.2, C49.1, C50.1, C51.1, C52.2, C53.2, C55.1, C56.1, C57.1, C58.1, C59.1, C60.1, C61.1, C63.1, D10.1 (A), D11.3 (GND), D12.1 (A), D18.3 (GND), D19.1 (A), D6.1 (A), D7.1 (A), D9.1 (A), J2.1 (S), J3.1 (S), J4.1 (S), J5.1 (S), J6.1 (S), J7.1, R31.2, R32.2, R33.2, R34.2, R48.2, R49.2, R53.2, R54.2, R59.2, R6.1, R67.1, R77.2, R80.2, R81.2, U15.4 (-VSS)
- net GNDD: now also U2.5 (ST), C1.2, C10.1, C16.1, C17.1, C19.2, C2.1, C20.2, C21.2, C22.1, C23.1, C24.2, C25.1, C26.2, C3.1, C4.1, C41.2, C42.2, C43.2, C44.2, C5.1, C6.1, C64.2, C7.1, C8.1, C9.1, D1.2 (A), R1.2, R12.2, R15.2, R16.2, R18.2, R2.1, R20.1, R24.1, R3.1, R6.2, R7.2, R78.2, R79.2, R8.2
- net G_CHG: now also R8.1, R9.1
- net G_DSG: now also R10.1, R11.1
- net LEDButton: now also R79.1
- net LightStimulus: now also R66.2
- net MISO: now also R43.2
- net MOSI: now also R41.1
- net Noise: now also C56.2, R63.2
- net PhotoDiode: now also C55.2, R62.2
- net PhotoGain: now also C51.2, R60.2
- net SCK: now also R42.1
- net Spike_BLED: now also R72.1
- net Spike_Buzzer: now also C62.1
- net Spike_GLED: now also R73.1
- net Spike_RLED: now also R74.1
- net Stim_BLED: now also R69.1
- net Stim_GLED: now also R70.1
- net Stim_RLED: now also R71.1
- net StimulusFrequency: now also C58.2, R65.2
- net StimulusStrength: now also C57.2, R64.2
- net Synapse1_Spike: now also D7.3, R51.2
- net Synapse2_Spike: now also D10.3, R56.2
- net SynapseGain1: now also U10.1 (CH0), C45.2, R47.2; no longer U10.3 (CH2)
- net SynapseGain2: now also U10.3 (CH2), C47.2, R52.2; no longer U10.1 (CH0)
- net SynapseIn1: now also U10.2 (CH1), C46.1, D6.3, R50.2; no longer U10.4 (CH3)
- net SynapseIn2: now also U10.4 (CH3), C48.1, D9.3, R55.2; no longer U10.2 (CH1)
- net SynapseOut: now also D17.1 (IO1), D18.1 (IO1), J6.3 (T), J7.3, R28.1, R80.1; no longer D17.2 (IO2)
- net SynapseOut_Spike: now also R76.1
- net USB_D+: now also R37.1
- net USB_D-: now also R36.1
- net VBUS: now also U5.1 (CE), U5.4 (VDD), C16.2, C2.2, C3.2, R17.2
- net VBUS_RAW: now also D1.1 (C)
- net VoltageMembrane: now also C49.2, R57.2
- net at Q3.1 (G): now also R23.2, R24.2
- net at D15.4 (BA): now also R69.2
- net at U12.14 (IO20): now also R37.2
- net +5VA: now reaches L3.2, U4.1 (IN), U4.3 (EN)
- net +5VA: now also C11.2, C12.2
- net at U12.19 (IO11): now also R41.2
- net at B1.1: now also C62.2
- net at D4.2: now also R22.2
- net at L5.1, U8.6 (VOUT): now also C26.1, R21.1, R22.1
- net at U12.17 (IO9): now also R39.2
- net at D14.1 (IO1): now also J5.2 (R), R68.2
- net at U6.5 (BAT): now also C18.2, R13.1
- net at D8.1 (IO1): now also J3.2 (R), R54.1, R56.1
- net at D13.2 (C), U13.2 (IN-): now also C54.1, R61.1
- net at U9.14 (VOUTA): now also R26.1
- net at D5.1 (IO1): now also J2.2 (R), R49.1, R51.1
- net at D5.2 (IO2): now also J2.3 (T), R48.1, R50.1
- net OscilloscopeStimulus: now reaches U11.4 (CH3)
- net OscilloscopeStimulus: now also C63.2, D19.3, R82.1
- net at U11.5 (CH4): now also R31.1
- net at U11.6 (CH5): now also R32.1
- net at U11.7 (CH6): now also R33.1
- net at U11.8 (CH7): now also R34.1
- net at D3.2: now also R5.1
- net at D8.2 (IO2): now also J3.3 (T), R53.1, R55.1
- net at D16.2 (BA): now also R72.2
- net at Q2.1 (G): now also R17.1, R18.1
- net at VR5.2: now also R63.1
- net at Q4.3 (D): now also D17.2 (IO2), J6.2 (R), R75.2; no longer D17.1 (IO1)
- net at U12.21 (IO13): now also R43.1
- net at L1.1, U2.6 (VOUT): now also C4.2
- net at Q4.1 (G): now also R76.2, R77.1
- net at U7.3 (L): now also L4.2
- net at VR3.2: now also R57.1
- net at U14.3 (IN+): now also C59.2, R66.1, R67.2
- net LightStimulus_Buff: now reaches U14.1 (OUT), U14.4 (IN-)
- net LightStimulus_Buff: now also R68.1
- net at U9.10 (VOUTB): now also R27.1
- net at U12.13 (IO19): now also R36.2
- net at VR2.2: now also R52.1
- net at VR7.2: now also R65.1
- net at VR1.2: now also R47.1
- net at D15.1 (RA): now also R71.2
- net at D15.3 (GA): now also R70.2
- net at U12.15 (IO3): now also R38.2
- net at U13.6 (OUT): now also C54.2, R61.2, R62.1
- net at VR6.2: now also R64.1
- net at U12.20 (IO12): now also R42.2
- net at VR4.2: now also R60.1
- net at D16.1 (RA): now also R74.2
- net at D16.3 (GA): now also R73.2
- net at U5.5 (PROG): now also R7.1
- net at D2.2: now also R4.1
- net at U8.5 (ST): now also R21.2, R23.1
- net at U6.6 (V-): now also R12.1
- net at U6.2 (COUT): now also R9.2
- net at U6.3 (DOUT): now also R11.2
- net at SW2.1 (A): now also R45.2
- net at U12.18 (IO10): now also R40.2
- new net: R29.1, U15.6 (-INB), U15.7 (OUTB)
- new net: R20.2, U7.8 (PS)
- new net: D18.2 (IO2), J7.2, R81.1, R82.2
- new net: D11.1 (IO1), J4.3 (T), R58.1, R59.1
- new net: R28.2, U15.1 (OUTA), U15.2 (-INA)
- new net CurrentStimulus_preBuff: R27.2, U15.5 (+INB)
- new net SynapseOut_preBuff: R26.2, U15.3 (+INA)
- no-connect marks 35 -> 29
Other:
- note added: "3.3 V Digital Rail Generation"
- note added: "5V Lines"
- note added: "Board power tree, source selection, battery management, control electronics, analogue acquisition and external signal interfaces. Distributes power from USB or battery operation and routes the front-panel controls, analogue readout and output signals to the main controller."
- note added: "Brings USB power and USB data onto the board. Provides the Type-C sink configuration, over-current protection and surge/ESD protection before VBUS and the USB data lines are passed into the rest of the system."
- note added: "Charges the single-cell LiPo battery from USB power using a dedicated charger IC. Sets the charge current, stabilises the charger supply. Generates the battery charge node used by the protected battery path."
- note added: "Combines the available 5 V sources into the main +5V rail while preventing reverse current between them. Forms the primary 5 V distribution node for the rest of the board. Isolates USB power from the battery-boosted supply."
- note added: "Converts the main +5V rail into the regulated +3.3V digital supply used by the controller and digital peripherals. Provides the main low-voltage logic rail for the board."
- note added: "ESP32-S3 WROOM1 N4"
- note added: "LiPo Cell Protection"
- note added: "Power, control and signal interface"
- note added: "Protects external connectors and user-accessible signal lines against ESD events and transient over-voltage. Reduces risk of damage or latch-up when cables are plugged, unplugged or mispatched."
- note added: "Protects the LiPo cell against over-charge, over-discharge and excessive current using a protection controller and back-to-back MOSFETs. Isolates the cell when unsafe operating conditions are detected."
- note added: "Spiky Oscilloscope Interface"
- note added: "Steps the protected battery voltage up to a regulated 5 V rail for stand-alone operation. Also includes the control network that allows the boost path to be enabled or inhibited depending on system power conditions."
- note added: "This section acquires the front-panel control associated with membrane voltage behaviour. It provides a stable analogue control value to the ADC so the firmware can adjust the neuron model accordingly."
- note added: "This section acquires the front-panel noise control used to vary the amount of injected or simulated noise in the system. It provides an adjustable analogue parameter for the controller."
- note added: "This section acquires the user controls associated with stimulus amplitude and timing and generates the corresponding stimulus-related signal path. It supports both front-panel parameter control and external stimulus output."
- note added: "This section conditions the first synapse input from the external connector before it is measured or interpreted by the controller. It includes the protection and biasing needed for robust front-panel patch use."
- note added: "This section conditions the second synapse input from the external connector before it is measured or interpreted by the controller. It mirrors the first synapse path to provide a second protected and measurable input channel."
- note added: "This section converts controller-generated digital values into analogue voltages and buffers them before they are sent to external outputs. It provides controlled low-impedance analogue drive for stimulus and related output signals."
- note added: "This section converts the photodiode current into a measurable voltage using an analogue front-end with gain and filtering. It provides the controller with a conditioned light-response signal."
- note added: "This section digitises the analogue control voltages and sensor signals used by the system. It provides the controller with measured values from the front-panel potentiometers and analogue inputs."
- note added: "This section drives the external synaptic output connector with the buffered output signal generated by the system. It provides a protected, low-impedance interface for patching the board to external equipment or other units."
- note added: "This section is the main digital controller of the board. It handles: USB communication Peripheral control Signal generation Data acquisition System coordination."
- note added: "This section routes selected internal signals to the external oscilloscope connection for monitoring and demonstration. It provides a convenient way to observe the generated waveforms and system activity on external instruments."
- note added: "USB-C entry"
- note removed: "ESP32S3 WROOM1 N4"
- note removed: "LiPo Battery Protection"
- note removed: "USB-C"
- note removed: "VOLTAGE REGULATOR"
- title: Spikeling v 3.1 -> Spikeling v 3.2
- moved on the sheet: B1, BT1, D13, D14, D15, D16, D17, D2, D3, D4, D5, D8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
