File: Hardware/PCB/Spikeling 3.2/Spikeling_v3.2.kicad_sch (KiCad schematic)
At the start: 219 parts, among them J1 Connector, USB-TYPE-C-16P, J2 Synapse1 In, J3 Synapse2 In, J4 Input Current, J5 Stimulus Out, J6 Synapse Out, J7 Oscilloscope Output, Q1 FS8205A, Q2 2N7002, Q3 2N7002, Q4 2N7002, SW1 K3-1260D-L1, SW2 Tactile Button, 160gf, SW3 SKHHLVA010, SW4 SKHHLVA010, SW5 SKHHLVA010, U1 MF-MSMF050-2, U10 MCP3208T-CI/SL, U11 MCP3208T-CI/SL, U12 ESP32-S3-WROOM-1-N4, U13 OPA380AIDGKR, U14 TLV9001IDBVR, U15 MCP6002T-I/SN, U2 LM66100DCKR, U3 TPS62162DSGR, U4 TPS7A2033PDBVR, U5 MCP73812T-420I/OT, U6 BQ29700DSER, U7 TPS61200DRCR, U8 LM66100DCKR, U9 MCP4922-E/SL

Commit message: update PCB
Parts:
- C15, C16, C17, C29, C31, C34, C38, C5, C52, C59: LCSC Part # C560882 -> C694229
- C22, C7: LCSC Part # C380364 -> C2171160
- D10, D12, D13, D19, D6, D7, D9, Q1, Q2, Q3, Q4, SW3, SW4, SW5, TV1, U13, U14, U4, U5: FT Rotation Offset (none) -> 180
- R11, R23, R26, R27, R45, R69, R70, R71, R72, R73, R74, R9: LCSC Part # C105588 -> C115420
- R14: LCSC Part # C23263 -> C2907075
- R28, R29: LCSC Part # C107696 -> C22962
- U10, U11, U15: FT Rotation Offset (none) -> 90
- U9: FT Rotation Offset (none) -> -90
